File: Data_Collection_KiCAD_Project/MEMS_ICM-20948.sch (KiCad schematic (older format))
At the start: 9 parts

Commit message: Schematic v1.0.4
Added I2C addresses to MEMS, Temp Sensor, and Barometer on main schematic page.
Other:
- note added: "ICM-20948 I2C Addresses:\nAD0 = 0 -> 0x68\nAD0 = 1 -> 0x69"
Changed lines of the file:
@@
 Title "ICM-20948 MEMS Chip"
 Date "2021-10-01"
-Rev "v1.0.3"
+Rev "v1.0.4"
 Comp "Missouri S&T Rocket Design Team '21 (Thomas Francois)"
 Comment1 "https://github.com/MSTRocketDesignTeam/Avionics-Data-Collection-PCB"
@@
 Text Notes 4800 4800 0    50   ~ 0
 LM317 Equation:\nVout = 1.25(1 + R2/R1)\nLet R1 = 240Ω, Vout = 1.8V\nR1 = 105.6Ω ≈ 100Ω
+Text Notes 7650 4500 0    50   ~ 0
+ICM-20948 I2C Addresses:\nAD0 = 0 -> 0x68\nAD0 = 1 -> 0x69
 $EndSCHEMATC
