File: Data_Collection_KiCAD_Project/Data_Collection_KiCAD_Project.sch (KiCad schematic (older format))
At the start: 3 parts

Commit message: Added Power Budget Spreadsheet
TODO:
-Implement I2C interrupt pin
-Add I2C Pullups
-Add I2C Capacitors
-Check for auxiliary pins needed from sensors
-Add power buffer cap and diode?
-Double check and finalize layouts
Parts:
- C?: symbol Device:C -> Data_Collection_KiCAD_Project-rescue:C-Device
Changed lines of the file:
@@
 $EndDescr
 $Comp
-L power:+5V #PWR?
+L Data_Collection_KiCAD_Project-rescue:+5V-power #PWR?
 U 1 1 61577BBB
 P 2400 6950
@@
 $EndComp
 $Comp
-L power:+3.3V #PWR?
+L Data_Collection_KiCAD_Project-rescue:+3.3V-power #PWR?
 U 1 1 61579C7C
 P 1200 6600
@@
 NoConn ~ 5450 7050
 $Comp
-L Device:C C?
+L Data_Collection_KiCAD_Project-rescue:C-Device C?
 U 1 1 619D380E
 P 5400 7350
@@
 $EndComp
 $Comp
-L power:GND #PWR?
+L Data_Collection_KiCAD_Project-rescue:GND-power #PWR?
 U 1 1 619D3F11
 P 5400 7500
@@
 NRST cap protects\nagainst parasitic resets.
 $Comp
-L power:GND #PWR?
+L Data_Collection_KiCAD_Project-rescue:GND-power #PWR?
 U 1 1 616E7AC6
 P 9400 1550
@@
 $EndComp
 $Comp
-L power:+3.3V #PWR?
+L Data_Collection_KiCAD_Project-rescue:+3.3V-power #PWR?
 U 1 1 616FEE96
 P 9400 1000
@@
 $EndComp
 $Comp
-L power:GND #PWR?
+L Data_Collection_KiCAD_Project-rescue:GND-power #PWR?
 U 1 1 6176C380
 P 7350 1550
@@
 	5500 2450 5500 2350
 $Comp
-L power:GND #PWR?
+L Data_Collection_KiCAD_Project-rescue:GND-power #PWR?
 U 1 1 617E2922
 P 5500 2450
@@
 	6150 6750 6150 6700
 $Comp
-L power:+3.3V #PWR?
+L Data_Collection_KiCAD_Project-rescue:+3.3V-power #PWR?
 U 1 1 619AF36E
 P 6150 6700
@@
 	6050 7200 6050 7150
 $Comp
-L power:GND #PWR?
+L Data_Collection_KiCAD_Project-rescue:GND-power #PWR?
 U 1 1 6196C349
 P 6050 7200
@@
 	1450 6900 1200 6900
 $Comp
-L power:GND #PWR?
+L Data_Collection_KiCAD_Project-rescue:GND-power #PWR?
 U 1 1 618118F6
 P 2200 7100
@@
 	1000 6800 1000 6950
 $Comp
-L power:GND #PWR?
+L Data_Collection_KiCAD_Project-rescue:GND-power #PWR?
 U 1 1 6181AAF8
 P 1000 6950
