File: Data_Collection_KiCAD_Project/Data_Collection_KiCAD_Project.sch (KiCad schematic (older format))
At the start: 0 parts

Commit message: Finalized Schematic
Parts:
- added TP1, TP2, TP3, TP4: Debug Pad, TestPoint:TestPoint_Plated_Hole_D2.0mm, symbol dk_Test-Points:RCT-0C
Connections:
- net BNO055/~BNO055_BTL: now also TP2.1
- net BNO055/~BNO055_RESET: now also TP1.1
- net KX134-1211/KX134_INT1: now also TP3.1
- net KX134-1211/KX134_INT2: now also TP4.1
Changed lines of the file:
@@
 Wire Wire Line
 	9650 1400 10150 1400
-$Sheet
-S 1550 5750 1150 1900
-U 619DD6DC
-F0 "Main Bus" 50
-F1 "file61A437B4.sch" 50
-F2 "t_mosi" I L 1550 5850 50
-F3 "t_miso" I L 1550 6000 50
-F4 "t_clk" I L 1550 6150 50
-F5 "Alert_scl" I L 1550 6350 50
-F6 "Alert_sda" I L 1550 6500 50
-F7 "Alert_Active" I L 1550 6650 50
-F8 "SWDIO" I L 1550 6850 50
-F9 "SWCLK" I L 1550 7000 50
-F10 "NRST" I L 1550 7150 50
-F11 "Fire" I L 1550 7350 50
-F12 "Fire_redundant" I L 1550 7500 50
-$EndSheet
 Entry Wire Line
 	1150 4600 1250 4500
@@
 Wire Wire Line
 	1250 4200 1550 4200
+$Sheet
+S 1550 5750 1150 1900
+U 619DD6DC
+F0 "Main Bus" 50
+F1 "DSUB.sch" 50
+F2 "t_mosi" I L 1550 5850 50
+F3 "t_miso" I L 1550 6000 50
+F4 "t_clk" I L 1550 6150 50
+F5 "Alert_scl" I L 1550 6350 50
+F6 "Alert_sda" I L 1550 6500 50
+F7 "Alert_Active" I L 1550 6650 50
+F8 "SWDIO" I L 1550 6850 50
+F9 "SWCLK" I L 1550 7000 50
+F10 "NRST" I L 1550 7150 50
+F11 "Fire" I L 1550 7350 50
+F12 "Fire_redundant" I L 1550 7500 50
+$EndSheet
+$Comp
+L dk_Test-Points:RCT-0C TP1
+U 1 1 61A7EB52
+P 4400 1150
+F 0 "TP1" V 4400 1050 50  0000 C CNN
+F 1 "Debug Pad" V 4266 1197 50  0001 C CNN
+F 2 "TestPoint:TestPoint_Plated_Hole_D2.0mm" H 4600 1350 60  0001 L CNN
+F 3 "https://www.te.com/commerce/DocumentDelivery/DDEController?Action=srchrtrv&DocNm=1773266&DocType=DS&DocLang=English" H 4600 1450 60  0001 L CNN
+F 4 "A106144CT-ND" H 4600 1550 60  0001 L CNN "Digi-Key_PN"
+F 5 "RCT-0C" H 4600 1650 60  0001 L CNN "MPN"
+F 6 "Test and Measurement" H 4600 1750 60  0001 L CNN "Category"
+F 7 "Test Points" H 4600 1850 60  0001 L CNN "Family"
+F 8 "https://www.te.com/commerce/DocumentDelivery/DDEController?Action=srchrtrv&DocNm=1773266&DocType=DS&DocLang=English" H 4600 1950 60  0001 L CNN "DK_Datasheet_Link"
+F 9 "/product-detail/en/te-connectivity-amp-connectors/RCT-0C/A106144CT-ND/3477801" H 4600 2050 60  0001 L CNN "DK_Detail_Page"
+F 10 "PC TEST POINT NATURAL" H 4600 2150 60  0001 L CNN "Description"
+F 11 "TE Connectivity AMP Connectors" H 4600 2250 60  0001 L CNN "Manufacturer"
+F 12 "Active" H 4600 2350 60  0001 L CNN "Status"
+	1    4400 1150
+	0    1    1    0
+$EndComp
+$Comp
+L dk_Test-Points:RCT-0C TP2
+U 1 1 61A84AF6
+P 4400 1300
+F 0 "TP2" V 4400 1200 50  0000 C CNN
+F 1 "Debug Pad" V 4266 1347 50  0001 C CNN
+F 2 "TestPoint:TestPoint_Plated_Hole_D2.0mm" H 4600 1500 60  0001 L CNN
+F 3 "https://www.te.com/commerce/DocumentDelivery/DDEController?Action=srchrtrv&DocNm=1773266&DocType=DS&DocLang=English" H 4600 1600 60  0001 L CNN
+F 4 "A106144CT-ND" H 4600 1700 60  0001 L CNN "Digi-Key_PN"
+F 5 "RCT-0C" H 4600 1800 60  0001 L CNN "MPN"
+F 6 "Test and Measurement" H 4600 1900 60  0001 L CNN "Category"
+F 7 "Test Points" H 4600 2000 60  0001 L CNN "Family"
+F 8 "https://www.te.com/commerce/DocumentDelivery/DDEController?Action=srchrtrv&DocNm=1773266&DocType=DS&DocLang=English" H 4600 2100 60  0001 L CNN "DK_Datasheet_Link"
+F 9 "/product-detail/en/te-connectivity-amp-connectors/RCT-0C/A106144CT-ND/3477801" H 4600 2200 60  0001 L CNN "DK_Detail_Page"
+F 10 "PC TEST POINT NATURAL" H 4600 2300 60  0001 L CNN "Description"
+F 11 "TE Connectivity AMP Connectors" H 4600 2400 60  0001 L CNN "Manufacturer"
+F 12 "Active" H 4600 2500 60  0001 L CNN "Status"
+	1    4400 1300
+	0    1    1    0
+$EndComp
+Wire Wire Line
+	4650 1150 4500 1150
+Wire Wire Line
+	4650 1300 4500 1300
+$Comp
+L dk_Test-Points:RCT-0C TP3
+U 1 1 61A8A234
+P 9950 1100
+F 0 "TP3" V 9950 1000 50  0000 C CNN
+F 1 "Debug Pad" V 9816 1147 50  0001 C CNN
+F 2 "TestPoint:TestPoint_Plated_Hole_D2.0mm" H 10150 1300 60  0001 L CNN
+F 3 "https://www.te.com/commerce/DocumentDelivery/DDEController?Action=srchrtrv&DocNm=1773266&DocType=DS&DocLang=English" H 10150 1400 60  0001 L CNN
+F 4 "A106144CT-ND" H 10150 1500 60  0001 L CNN "Digi-Key_PN"
+F 5 "RCT-0C" H 10150 1600 60  0001 L CNN "MPN"
+F 6 "Test and Measurement" H 10150 1700 60  0001 L CNN "Category"
+F 7 "Test Points" H 10150 1800 60  0001 L CNN "Family"
+F 8 "https://www.te.com/commerce/DocumentDelivery/DDEController?Action=srchrtrv&DocNm=1773266&DocType=DS&DocLang=English" H 10150 1900 60  0001 L CNN "DK_Datasheet_Link"
+F 9 "/product-detail/en/te-connectivity-amp-connectors/RCT-0C/A106144CT-ND/3477801" H 10150 2000 60  0001 L CNN "DK_Detail_Page"
+F 10 "PC TEST POINT NATURAL" H 10150 2100 60  0001 L CNN "Description"
+F 11 "TE Connectivity AMP Connectors" H 10150 2200 60  0001 L CNN "Manufacturer"
+F 12 "Active" H 10150 2300 60  0001 L CNN "Status"
+	1    9950 1100
+	0    1    1    0
+$EndComp
+$Comp
+L dk_Test-Points:RCT-0C TP4
+U 1 1 61A902C0
+P 9950 1250
+F 0 "TP4" V 9950 1150 50  0000 C CNN
+F 1 "Debug Pad" V 9816 1297 50  0001 C CNN
+F 2 "TestPoint:TestPoint_Plated_Hole_D2.0mm" H 10150 1450 60  0001 L CNN
+F 3 "https://www.te.com/commerce/DocumentDelivery/DDEController?Action=srchrtrv&DocNm=1773266&DocType=DS&DocLang=English" H 10150 1550 60  0001 L CNN
+F 4 "A106144CT-ND" H 10150 1650 60  0001 L CNN "Digi-Key_PN"
+F 5 "RCT-0C" H 10150 1750 60  0001 L CNN "MPN"
+F 6 "Test and Measurement" H 10150 1850 60  0001 L CNN "Category"
+F 7 "Test Points" H 10150 1950 60  0001 L CNN "Family"
+F 8 "https://www.te.com/commerce/DocumentDelivery/DDEController?Action=srchrtrv&DocNm=1773266&DocType=DS&DocLang=English" H 10150 2050 60  0001 L CNN "DK_Datasheet_Link"
+F 9 "/product-detail/en/te-connectivity-amp-connectors/RCT-0C/A106144CT-ND/3477801" H 10150 2150 60  0001 L CNN "DK_Detail_Page"
+F 10 "PC TEST POINT NATURAL" H 10150 2250 60  0001 L CNN "Description"
+F 11 "TE Connectivity AMP Connectors" H 10150 2350 60  0001 L CNN "Manufacturer"
+F 12 "Active" H 10150 2450 60  0001 L CNN "Status"
+	1    9950 1250
+	0    1    1    0
+$EndComp
+Wire Wire Line
+	10150 1100 10050 1100
+Wire Wire Line
+	10150 1250 10050 1250
 Wire Bus Line
 	3250 1700 3250 1900

Commit message: Changed MCU and started pcb
Parts:
- TP1, TP2, TP3, TP4: footprint TestPoint:TestPoint_Plated_Hole_D2.0mm -> TestPoint:TestPoint_Pad_D1.0mm
Changed lines of the file:
@@
 Wire Wire Line
 	8050 1800 8050 1250
-$Sheet
-S 1550 1450 1000 4050
-U 61E8EFE4
-F0 "L552CC" 50
-F1 "MCU_L552CC.sch" 50
-F2 "I2C1_SCL" I R 2550 1750 50
-F3 "I2C1_SDA" I R 2550 1600 50
-F4 "SPI2_SCK" I L 1550 3700 50
-F5 "SPI2_MISO" I L 1550 3500 50
-F6 "SPI2_MOSI" I L 1550 3900 50
-F7 "SPI1_SCK" I R 2550 2650 50
-F8 "USART2_TX" I R 2550 4150 50
-F9 "USART2_RX" I R 2550 4000 50
-F10 "SPI1_MISO" I R 2550 2950 50
-F11 "SPI1_MOSI" I R 2550 2800 50
-F12 "USB_DM" I R 2550 5350 50
-F13 "USB_DP" I R 2550 5200 50
-F14 "SWDIO" I L 1550 5350 50
-F15 "SWCLK" I L 1550 5200 50
-F16 "NRST" I L 1550 5050 50
-F17 "PVD_IN" I L 1550 4850 50
-F18 "EXT_SDA" I L 1550 4500 50
-F19 "EXT_SCL" I L 1550 4350 50
-F20 "EXT_I2C_Alert" B L 1550 4200 50
-$EndSheet
 Wire Wire Line
 	5500 2350 5350 2350
@@
 Text Label 1550 6000 2    50   ~ 0
 SPI2_MISO
-Text Label 1600 6150 2    50   ~ 0
+Text Label 1550 6150 2    50   ~ 0
 SPI2_SCK
 Text Label 1550 5850 2    50   ~ 0
@@
 F2 "t_mosi" I L 1550 5850 50
 F3 "t_miso" I L 1550 6000 50
-F4 "t_clk" I L 1550 6150 50
-F5 "Alert_scl" I L 1550 6350 50
-F6 "Alert_sda" I L 1550 6500 50
-F7 "Alert_Active" I L 1550 6650 50
-F8 "SWDIO" I L 1550 6850 50
-F9 "SWCLK" I L 1550 7000 50
-F10 "NRST" I L 1550 7150 50
-F11 "Fire" I L 1550 7350 50
-F12 "Fire_redundant" I L 1550 7500 50
+F4 "Alert_scl" I L 1550 6350 50
+F5 "Alert_sda" I L 1550 6500 50
+F6 "Alert_Active" I L 1550 6650 50
+F7 "SWDIO" I L 1550 6850 50
+F8 "SWCLK" I L 1550 7000 50
+F9 "NRST" I L 1550 7150 50
+F10 "Fire" I L 1550 7350 50
+F11 "Fire_redundant" I L 1550 7500 50
+F12 "t_clk" I L 1550 6150 50
 $EndSheet
 $Comp
@@
 F 0 "TP1" V 4400 1050 50  0000 C CNN
 F 1 "Debug Pad" V 4266 1197 50  0001 C CNN
-F 2 "TestPoint:TestPoint_Plated_Hole_D2.0mm" H 4600 1350 60  0001 L CNN
+F 2 "TestPoint:TestPoint_Pad_D1.0mm" H 4600 1350 60  0001 L CNN
 F 3 "https://www.te.com/commerce/DocumentDelivery/DDEController?Action=srchrtrv&DocNm=1773266&DocType=DS&DocLang=English" H 4600 1450 60  0001 L CNN
 F 4 "A106144CT-ND" H 4600 1550 60  0001 L CNN "Digi-Key_PN"
@@
 F 0 "TP2" V 4400 1200 50  0000 C CNN
 F 1 "Debug Pad" V 4266 1347 50  0001 C CNN
-F 2 "TestPoint:TestPoint_Plated_Hole_D2.0mm" H 4600 1500 60  0001 L CNN
+F 2 "TestPoint:TestPoint_Pad_D1.0mm" H 4600 1500 60  0001 L CNN
 F 3 "https://www.te.com/commerce/DocumentDelivery/DDEController?Action=srchrtrv&DocNm=1773266&DocType=DS&DocLang=English" H 4600 1600 60  0001 L CNN
 F 4 "A106144CT-ND" H 4600 1700 60  0001 L CNN "Digi-Key_PN"
@@
 F 0 "TP3" V 9950 1000 50  0000 C CNN
 F 1 "Debug Pad" V 9816 1147 50  0001 C CNN
-F 2 "TestPoint:TestPoint_Plated_Hole_D2.0mm" H 10150 1300 60  0001 L CNN
+F 2 "TestPoint:TestPoint_Pad_D1.0mm" H 10150 1300 60  0001 L CNN
 F 3 "https://www.te.com/commerce/DocumentDelivery/DDEController?Action=srchrtrv&DocNm=1773266&DocType=DS&DocLang=English" H 10150 1400 60  0001 L CNN
 F 4 "A106144CT-ND" H 10150 1500 60  0001 L CNN "Digi-Key_PN"
@@
 F 0 "TP4" V 9950 1150 50  0000 C CNN
 F 1 "Debug Pad" V 9816 1297 50  0001 C CNN
-F 2 "TestPoint:TestPoint_Plated_Hole_D2.0mm" H 10150 1450 60  0001 L CNN
+F 2 "TestPoint:TestPoint_Pad_D1.0mm" H 10150 1450 60  0001 L CNN
 F 3 "https://www.te.com/commerce/DocumentDelivery/DDEController?Action=srchrtrv&DocNm=1773266&DocType=DS&DocLang=English" H 10150 1550 60  0001 L CNN
 F 4 "A106144CT-ND" H 10150 1650 60  0001 L CNN "Digi-Key_PN"
@@
 Wire Wire Line
 	10150 1250 10050 1250
+$Sheet
+S 1550 1450 1000 4050
+U 61E8EFE4
+F0 "L552CC" 50
+F1 "MCU_STM32L562VET6Q.sch" 50
+F2 "I2C1_SCL" I R 2550 1750 50
+F3 "I2C1_SDA" I R 2550 1600 50
+F4 "SPI2_SCK" I L 1550 3700 50
+F5 "SPI2_MISO" I L 1550 3500 50
+F6 "SPI2_MOSI" I L 1550 3900 50
+F7 "SPI1_SCK" I R 2550 2650 50
+F8 "USART2_TX" I R 2550 4150 50
+F9 "USART2_RX" I R 2550 4000 50
+F10 "SPI1_MISO" I R 2550 2950 50
+F11 "SPI1_MOSI" I R 2550 2800 50
+F12 "USB_DM" I R 2550 5350 50
+F13 "USB_DP" I R 2550 5200 50
+F14 "SWDIO" I L 1550 5350 50
+F15 "SWCLK" I L 1550 5200 50
+F16 "NRST" I L 1550 5050 50
+F17 "EXT_SDA" I L 1550 4500 50
+F18 "EXT_SCL" I L 1550 4350 50
+F19 "EXT_I2C_Alert" B L 1550 4200 50
+$EndSheet
 Wire Bus Line
 	3250 1700 3250 1900

Commit message: progress update
Parts:
- TP1, TP2, TP3, TP4: footprint TestPoint:TestPoint_Pad_D1.0mm -> Connector_PinHeader_1.00mm:PinHeader_1x01_P1.00mm_Vertical
Changed lines of the file:
@@
 F 0 "TP1" V 4400 1050 50  0000 C CNN
 F 1 "Debug Pad" V 4266 1197 50  0001 C CNN
-F 2 "TestPoint:TestPoint_Pad_D1.0mm" H 4600 1350 60  0001 L CNN
+F 2 "Connector_PinHeader_1.00mm:PinHeader_1x01_P1.00mm_Vertical" H 4600 1350 60  0001 L CNN
 F 3 "https://www.te.com/commerce/DocumentDelivery/DDEController?Action=srchrtrv&DocNm=1773266&DocType=DS&DocLang=English" H 4600 1450 60  0001 L CNN
 F 4 "A106144CT-ND" H 4600 1550 60  0001 L CNN "Digi-Key_PN"
@@
 F 0 "TP2" V 4400 1200 50  0000 C CNN
 F 1 "Debug Pad" V 4266 1347 50  0001 C CNN
-F 2 "TestPoint:TestPoint_Pad_D1.0mm" H 4600 1500 60  0001 L CNN
+F 2 "Connector_PinHeader_1.00mm:PinHeader_1x01_P1.00mm_Vertical" H 4600 1500 60  0001 L CNN
 F 3 "https://www.te.com/commerce/DocumentDelivery/DDEController?Action=srchrtrv&DocNm=1773266&DocType=DS&DocLang=English" H 4600 1600 60  0001 L CNN
 F 4 "A106144CT-ND" H 4600 1700 60  0001 L CNN "Digi-Key_PN"
@@
 F 0 "TP3" V 9950 1000 50  0000 C CNN
 F 1 "Debug Pad" V 9816 1147 50  0001 C CNN
-F 2 "TestPoint:TestPoint_Pad_D1.0mm" H 10150 1300 60  0001 L CNN
+F 2 "Connector_PinHeader_1.00mm:PinHeader_1x01_P1.00mm_Vertical" H 10150 1300 60  0001 L CNN
 F 3 "https://www.te.com/commerce/DocumentDelivery/DDEController?Action=srchrtrv&DocNm=1773266&DocType=DS&DocLang=English" H 10150 1400 60  0001 L CNN
 F 4 "A106144CT-ND" H 10150 1500 60  0001 L CNN "Digi-Key_PN"
@@
 F 0 "TP4" V 9950 1150 50  0000 C CNN
 F 1 "Debug Pad" V 9816 1297 50  0001 C CNN
-F 2 "TestPoint:TestPoint_Pad_D1.0mm" H 10150 1450 60  0001 L CNN
+F 2 "Connector_PinHeader_1.00mm:PinHeader_1x01_P1.00mm_Vertical" H 10150 1450 60  0001 L CNN
 F 3 "https://www.te.com/commerce/DocumentDelivery/DDEController?Action=srchrtrv&DocNm=1773266&DocType=DS&DocLang=English" H 10150 1550 60  0001 L CNN
 F 4 "A106144CT-ND" H 10150 1650 60  0001 L CNN "Digi-Key_PN"
