File: Data_Collection_KiCAD_Project/FLASH_W25Q32JV.sch (KiCad schematic (older format))
At the start: 2 parts

Commit message: Added Power Budget Spreadsheet
TODO:
-Implement I2C interrupt pin
-Add I2C Pullups
-Add I2C Capacitors
-Check for auxiliary pins needed from sensors
-Add power buffer cap and diode?
-Double check and finalize layouts
Parts:
- C?: symbol Device:C -> Data_Collection_KiCAD_Project-rescue:C-Device
- U?: symbol Memory_Flash:W25Q32JVSS -> Data_Collection_KiCAD_Project-rescue:W25Q32JVSS-Memory_Flash
Changed lines of the file:
@@
 $EndDescr
 $Comp
-L power:+3.3V #PWR?
+L Data_Collection_KiCAD_Project-rescue:+3.3V-power #PWR?
 U 1 1 6161184E
 P 4150 2700
@@
 	4950 2800 4950 2750
 $Comp
-L power:GND #PWR?
+L Data_Collection_KiCAD_Project-rescue:GND-power #PWR?
 U 1 1 61611855
 P 4950 3600
@@
 Flash Storage Chip
 $Comp
-L Device:C C?
+L Data_Collection_KiCAD_Project-rescue:C-Device C?
 U 1 1 6161186E
 P 3850 3150
@@
 ~CS
 $Comp
-L Memory_Flash:W25Q32JVSS U?
+L Data_Collection_KiCAD_Project-rescue:W25Q32JVSS-Memory_Flash U?
 U 1 1 61611848
 P 4950 3200
@@
 $EndComp
 $Comp
-L power:GND #PWR?
+L Data_Collection_KiCAD_Project-rescue:GND-power #PWR?
 U 1 1 617DF3FC
 P 5500 3450
@@
 Connection ~ 5500 3400
 $Comp
-L power:GND #PWR?
+L Data_Collection_KiCAD_Project-rescue:GND-power #PWR?
 U 1 1 617DFAF5
 P 3850 3300
