File: Data_Collection_KiCAD_Project/GNSS_MAX-8Q.sch (KiCad schematic (older format))
At the start: 13 parts

Commit message: Added Power Budget Spreadsheet
TODO:
-Implement I2C interrupt pin
-Add I2C Pullups
-Add I2C Capacitors
-Check for auxiliary pins needed from sensors
-Add power buffer cap and diode?
-Double check and finalize layouts
Parts:
- C? (x6): symbol Device:C -> Data_Collection_KiCAD_Project-rescue:C-Device
- J?: symbol Connector:Conn_Coaxial -> Data_Collection_KiCAD_Project-rescue:Conn_Coaxial-Connector
- L?: symbol Device:L -> Data_Collection_KiCAD_Project-rescue:L-Device
- Q?: symbol Transistor_FET:FDC6330L -> Data_Collection_KiCAD_Project-rescue:FDC6330L-Transistor_FET
- R? (x3): symbol Device:R -> Data_Collection_KiCAD_Project-rescue:R-Device
- U?: symbol RF_GPS:MAX-8Q -> Data_Collection_KiCAD_Project-rescue:MAX-8Q-RF_GPS
Changed lines of the file:
@@
 $EndDescr
 $Comp
-L Device:L L?
+L Data_Collection_KiCAD_Project-rescue:L-Device L?
 U 1 1 616192D0
 P 3650 5950
@@
 $EndComp
 $Comp
-L power:GND #PWR?
+L Data_Collection_KiCAD_Project-rescue:GND-power #PWR?
 U 1 1 616192D6
 P 4000 6500
@@
 $EndComp
 $Comp
-L Device:C C?
+L Data_Collection_KiCAD_Project-rescue:C-Device C?
 U 1 1 616192DC
 P 4900 5550
@@
 $EndComp
 $Comp
-L Device:R R?
+L Data_Collection_KiCAD_Project-rescue:R-Device R?
 U 1 1 616192E2
 P 4700 5550
@@
 $EndComp
 $Comp
-L Device:R R?
+L Data_Collection_KiCAD_Project-rescue:R-Device R?
 U 1 1 616192E8
 P 4350 6250
@@
 $EndComp
 $Comp
-L Transistor_FET:FDC6330L Q?
+L Data_Collection_KiCAD_Project-rescue:FDC6330L-Transistor_FET Q?
 U 1 1 616192EF
 P 4000 5650
@@
 Connection ~ 4700 5350
 $Comp
-L power:GND #PWR?
+L Data_Collection_KiCAD_Project-rescue:GND-power #PWR?
 U 1 1 616192FE
 P 4900 5750
@@
 Connection ~ 4900 5350
 $Comp
-L Device:R R?
+L Data_Collection_KiCAD_Project-rescue:R-Device R?
 U 1 1 61619311
 P 3650 5550
@@
 	5500 6750 3000 6750
 $Comp
-L power:+3.3V #PWR?
+L Data_Collection_KiCAD_Project-rescue:+3.3V-power #PWR?
 U 1 1 6161C95B
 P 7200 2400
@@
 Connection ~ 7600 2450
 $Comp
-L power:GND #PWR?
+L Data_Collection_KiCAD_Project-rescue:GND-power #PWR?
 U 1 1 6161C967
 P 7700 3900
@@
 Connection ~ 7500 2450
 $Comp
-L Connector:Conn_Coaxial J?
+L Data_Collection_KiCAD_Project-rescue:Conn_Coaxial-Connector J?
 U 1 1 6161C976
 P 9400 3200
@@
 MAX-8Q: GNSS Module Chip
 $Comp
-L power:GND #PWR?
+L Data_Collection_KiCAD_Project-rescue:GND-power #PWR?
 U 1 1 6161C998
 P 1200 1950
@@
 $EndComp
 $Comp
-L Device:C C?
+L Data_Collection_KiCAD_Project-rescue:C-Device C?
 U 1 1 6161C99E
 P 1200 1700
@@
 $EndComp
 $Comp
-L power:+3.3V #PWR?
+L Data_Collection_KiCAD_Project-rescue:+3.3V-power #PWR?
 U 1 1 6161C9A4
 P 1200 1450
@@
 	1200 1450 1200 1500
 $Comp
-L Device:C C?
+L Data_Collection_KiCAD_Project-rescue:C-Device C?
 U 1 1 6161C9AC
 P 1600 1700
@@
 $EndComp
 $Comp
-L Device:C C?
+L Data_Collection_KiCAD_Project-rescue:C-Device C?
 U 1 1 6161C9B2
 P 2050 1700
@@
 $EndComp
 $Comp
-L Device:C C?
+L Data_Collection_KiCAD_Project-rescue:C-Device C?
 U 1 1 6161C9B8
 P 2500 1700
@@
 	1600 1900 2050 1900
 $Comp
-L Device:C C?
+L Data_Collection_KiCAD_Project-rescue:C-Device C?
 U 1 1 6161C9D2
 P 2950 1700
@@
 GPS_LNA_EN
 $Comp
-L power:GND #PWR?
+L Data_Collection_KiCAD_Project-rescue:GND-power #PWR?
 U 1 1 61679BC7
 P 9400 3400
@@
 ~RESET
 $Comp
-L power:GND #PWR?
+L Data_Collection_KiCAD_Project-rescue:GND-power #PWR?
 U 1 1 6167BBB2
 P 6550 3700
@@
 	6550 3400 7100 3400
 $Comp
-L RF_GPS:MAX-8Q U?
+L Data_Collection_KiCAD_Project-rescue:MAX-8Q-RF_GPS U?
 U 1 1 6161C986
 P 7700 3200
