File: Data_Collection_KiCAD_Project/MCU_L552CC.sch (KiCad schematic (older format))
At the start: 12 parts

Commit message: Formatting
Misc Formatting and CubeIDE configuration.
Also Added datasheets folder
Connections:
- net MEMS_EN: no longer names the net of U?.18 (PB0)
Changed lines of the file:
@@
 Text Notes 750  2400 0    50   ~ 0
 PVD_IN is the Power Voltage Dropout pin,\nused to detect and respond to brownout conditions.
-Text HLabel 8200 4200 0    50   Input ~ 0
-MEMS_EN
 Text HLabel 8200 4800 0    50   Input ~ 0
 I2C1_SCL

Commit message: Added Power Budget Spreadsheet
TODO:
-Implement I2C interrupt pin
-Add I2C Pullups
-Add I2C Capacitors
-Check for auxiliary pins needed from sensors
-Add power buffer cap and diode?
-Double check and finalize layouts
Parts:
- C? (x7): symbol Device:C -> Data_Collection_KiCAD_Project-rescue:C-Device
- D? (x3): symbol Device:LED -> Data_Collection_KiCAD_Project-rescue:LED-Device
- U?: symbol MCU_ST_STM32L0:STM32L031C4Tx -> Data_Collection_KiCAD_Project-rescue:STM32L031C4Tx-MCU_ST_STM32L0
- Y?: symbol Device:Crystal -> Data_Collection_KiCAD_Project-rescue:Crystal-Device
Changed lines of the file:
@@
 $EndDescr
 $Comp
-L MCU_ST_STM32L0:STM32L031C4Tx U?
+L Data_Collection_KiCAD_Project-rescue:STM32L031C4Tx-MCU_ST_STM32L0 U?
 U 1 1 61E9E6C0
 P 8800 4300
@@
 $EndComp
 $Comp
-L power:GND #PWR?
+L Data_Collection_KiCAD_Project-rescue:GND-power #PWR?
 U 1 1 61E9E6C6
 P 8700 6000
@@
 	8800 5950 8900 5950
 $Comp
-L power:+3.3V #PWR?
+L Data_Collection_KiCAD_Project-rescue:+3.3V-power #PWR?
 U 1 1 61E9E6D6
 P 9200 2700
@@
 Microcontroller Chip
 $Comp
-L power:GND #PWR?
+L Data_Collection_KiCAD_Project-rescue:GND-power #PWR?
 U 1 1 61E9E6FD
 P 6700 3300
@@
 NoConn ~ 9400 4200
 $Comp
-L Device:LED D?
+L Data_Collection_KiCAD_Project-rescue:LED-Device D?
 U 1 1 61E9E710
 P 9950 5300
@@
 $EndComp
 $Comp
-L Device:LED D?
+L Data_Collection_KiCAD_Project-rescue:LED-Device D?
 U 1 1 61E9E716
 P 10300 5300
@@
 $EndComp
 $Comp
-L Device:LED D?
+L Data_Collection_KiCAD_Project-rescue:LED-Device D?
 U 1 1 61E9E71C
 P 10650 5300
@@
 	9950 5000 9400 5000
 $Comp
-L power:GND #PWR?
+L Data_Collection_KiCAD_Project-rescue:GND-power #PWR?
 U 1 1 61E9E724
 P 9950 5450
@@
 $EndComp
 $Comp
-L power:GND #PWR?
+L Data_Collection_KiCAD_Project-rescue:GND-power #PWR?
 U 1 1 61E9E72A
 P 10300 5450
@@
 $EndComp
 $Comp
-L power:GND #PWR?
+L Data_Collection_KiCAD_Project-rescue:GND-power #PWR?
 U 1 1 61E9E730
 P 10650 5450
@@
 CL = 2 * (Cload - Cstray)\nCstray ≈ 20pF, Cstray ≈ 5pF\nCL = 2 * (Cload - 5pF)\nCL = 30pF
 $Comp
-L Device:Crystal Y?
+L Data_Collection_KiCAD_Project-rescue:Crystal-Device Y?
 U 1 1 61E9E73C
 P 7100 4300
@@
 $EndComp
 $Comp
-L Device:C C?
+L Data_Collection_KiCAD_Project-rescue:C-Device C?
 U 1 1 61E9E742
 P 6850 4650
@@
 $EndComp
 $Comp
-L Device:C C?
+L Data_Collection_KiCAD_Project-rescue:C-Device C?
 U 1 1 61E9E748
 P 7350 4650
@@
 	7350 4300 7250 4300
 $Comp
-L power:GND #PWR?
+L Data_Collection_KiCAD_Project-rescue:GND-power #PWR?
 U 1 1 61E9E750
 P 6850 4800
@@
 $EndComp
 $Comp
-L power:GND #PWR?
+L Data_Collection_KiCAD_Project-rescue:GND-power #PWR?
 U 1 1 61E9E756
 P 7350 4800
@@
 	6850 3400 6850 4300
 $Comp
-L power:GND #PWR?
+L Data_Collection_KiCAD_Project-rescue:GND-power #PWR?
 U 1 1 61EA2645
 P 900 1700
@@
 $EndComp
 $Comp
-L Device:C C?
+L Data_Collection_KiCAD_Project-rescue:C-Device C?
 U 1 1 61EA264B
 P 900 1450
@@
 $EndComp
 $Comp
-L power:+3.3V #PWR?
+L Data_Collection_KiCAD_Project-rescue:+3.3V-power #PWR?
 U 1 1 61EA2651
 P 900 1200
@@
 	900  1200 900  1250
 $Comp
-L Device:C C?
+L Data_Collection_KiCAD_Project-rescue:C-Device C?
 U 1 1 61EA2659
 P 1300 1450
@@
 $EndComp
 $Comp
-L Device:C C?
+L Data_Collection_KiCAD_Project-rescue:C-Device C?
 U 1 1 61EA265F
 P 1750 1450
@@
 $EndComp
 $Comp
-L Device:C C?
+L Data_Collection_KiCAD_Project-rescue:C-Device C?
 U 1 1 61EA2665
 P 2200 1450
@@
 	1300 1650 1750 1650
 $Comp
-L Device:C C?
+L Data_Collection_KiCAD_Project-rescue:C-Device C?
 U 1 1 61EA267F
 P 2650 1450
