File: Data_Collection_KiCAD_Project/MEMS_BNO055.sch (KiCad schematic (older format))
At the start: 6 parts

Commit message: Added Power Budget Spreadsheet
TODO:
-Implement I2C interrupt pin
-Add I2C Pullups
-Add I2C Capacitors
-Check for auxiliary pins needed from sensors
-Add power buffer cap and diode?
-Double check and finalize layouts
Parts:
- C? (x4): symbol Device:C_Small -> Data_Collection_KiCAD_Project-rescue:C_Small-Device
- U?: symbol Sensor_Motion:BNO055 -> Data_Collection_KiCAD_Project-rescue:BNO055-Sensor_Motion
- Y?: symbol Device:Crystal_Small -> Data_Collection_KiCAD_Project-rescue:Crystal_Small-Device
Changed lines of the file:
@@
 $EndDescr
 $Comp
-L Sensor_Motion:BNO055 U?
+L Data_Collection_KiCAD_Project-rescue:BNO055-Sensor_Motion U?
 U 1 1 61663BA8
 P 5650 3550
@@
 	5750 2700 5550 2700
 $Comp
-L power:+3.3V #PWR?
+L Data_Collection_KiCAD_Project-rescue:+3.3V-power #PWR?
 U 1 1 6166AFE6
 P 5200 2700
@@
 Connection ~ 5550 2700
 $Comp
-L power:GND #PWR?
+L Data_Collection_KiCAD_Project-rescue:GND-power #PWR?
 U 1 1 6166C199
 P 6400 2750
@@
 $EndComp
 $Comp
-L power:GND #PWR?
+L Data_Collection_KiCAD_Project-rescue:GND-power #PWR?
 U 1 1 6166D1D4
 P 5550 4350
@@
 ~BNO055_BTL
 $Comp
-L Device:Crystal_Small Y?
+L Data_Collection_KiCAD_Project-rescue:Crystal_Small-Device Y?
 U 1 1 6166FF64
 P 6450 3300
@@
 $EndComp
 $Comp
-L Device:C_Small C?
+L Data_Collection_KiCAD_Project-rescue:C_Small-Device C?
 U 1 1 6167196C
 P 6300 2700
@@
 	6450 3050 6450 3200
 $Comp
-L Device:C_Small C?
+L Data_Collection_KiCAD_Project-rescue:C_Small-Device C?
 U 1 1 6167A718
 P 6750 3050
@@
 $EndComp
 $Comp
-L Device:C_Small C?
+L Data_Collection_KiCAD_Project-rescue:C_Small-Device C?
 U 1 1 6167C82F
 P 6750 3550
@@
 Connection ~ 6450 3050
 $Comp
-L power:GND #PWR?
+L Data_Collection_KiCAD_Project-rescue:GND-power #PWR?
 U 1 1 6167EB61
 P 7100 3550
@@
 SCL
 $Comp
-L power:GND #PWR?
+L Data_Collection_KiCAD_Project-rescue:GND-power #PWR?
 U 1 1 61681CEA
 P 4850 4100
@@
 BNO055_INT
 $Comp
-L power:GND #PWR?
+L Data_Collection_KiCAD_Project-rescue:GND-power #PWR?
 U 1 1 616939D5
 P 6700 4350
@@
 $EndComp
 $Comp
-L Device:C_Small C?
+L Data_Collection_KiCAD_Project-rescue:C_Small-Device C?
 U 1 1 616964F3
 P 6450 4050
