File: Data_Collection_KiCAD_Project/MEMS_KX134.sch (KiCad schematic (older format))
At the start: 2 parts

Commit message: Added Power Budget Spreadsheet
TODO:
-Implement I2C interrupt pin
-Add I2C Pullups
-Add I2C Capacitors
-Check for auxiliary pins needed from sensors
-Add power buffer cap and diode?
-Double check and finalize layouts
Parts:
- C?: symbol Device:C_Small -> Data_Collection_KiCAD_Project-rescue:C_Small-Device
- U?: symbol Sensor_Motion:KX122-1042 -> Data_Collection_KiCAD_Project-rescue:KX122-1042-Sensor_Motion
Changed lines of the file:
@@
 $EndDescr
 $Comp
-L Sensor_Motion:KX122-1042 U?
+L Data_Collection_KiCAD_Project-rescue:KX122-1042-Sensor_Motion U?
 U 1 1 6165C3D0
 P 5950 3450
@@
 SCL
 $Comp
-L power:GND #PWR?
+L Data_Collection_KiCAD_Project-rescue:GND-power #PWR?
 U 1 1 61692503
 P 5950 3950
@@
 $EndComp
 $Comp
-L power:+3.3V #PWR?
+L Data_Collection_KiCAD_Project-rescue:+3.3V-power #PWR?
 U 1 1 6169CC30
 P 5350 2900
@@
 $EndComp
 $Comp
-L Device:C_Small C?
+L Data_Collection_KiCAD_Project-rescue:C_Small-Device C?
 U 1 1 6169DA95
 P 6450 2900
@@
 $EndComp
 $Comp
-L power:GND #PWR?
+L Data_Collection_KiCAD_Project-rescue:GND-power #PWR?
 U 1 1 6169E39E
 P 6650 2900
@@
 KX134-1211 I2C Addresses:\nADDR = 0 -> 0x1E\nADDR = 1 -> 0x1F
 $Comp
-L power:GND #PWR?
+L Data_Collection_KiCAD_Project-rescue:GND-power #PWR?
 U 1 1 616ACA8D
 P 5200 3600
@@
 	5200 3450 5200 3600
 $Comp
-L power:GND #PWR?
+L Data_Collection_KiCAD_Project-rescue:GND-power #PWR?
 U 1 1 616AF0ED
 P 6700 3900
