File: Data_Collection_KiCAD_Project/USB_ESD.sch (KiCad schematic (older format))
At the start: 12 parts

Commit message: Added Power Budget Spreadsheet
TODO:
-Implement I2C interrupt pin
-Add I2C Pullups
-Add I2C Capacitors
-Check for auxiliary pins needed from sensors
-Add power buffer cap and diode?
-Double check and finalize layouts
Parts:
- C? (x2): symbol Device:C -> Data_Collection_KiCAD_Project-rescue:C-Device
- D?: symbol Device:LED -> Data_Collection_KiCAD_Project-rescue:LED-Device
- D? (x2): symbol Device:D_Zener -> Data_Collection_KiCAD_Project-rescue:D_Zener-Device
- FB?: symbol Device:Ferrite_Bead_Small -> Data_Collection_KiCAD_Project-rescue:Ferrite_Bead_Small-Device
- J?: symbol Connector:USB_B_Micro -> Data_Collection_KiCAD_Project-rescue:USB_B_Micro-Connector
- R? (x3): symbol Device:R -> Data_Collection_KiCAD_Project-rescue:R-Device
- U?: symbol Power_Protection:USBLC6-2SC6 -> Data_Collection_KiCAD_Project-rescue:USBLC6-2SC6-Power_Protection
Changed lines of the file:
@@
 $EndDescr
 $Comp
-L Connector:USB_B_Micro J?
+L Data_Collection_KiCAD_Project-rescue:USB_B_Micro-Connector J?
 U 1 1 616146B0
 P 2150 3950
@@
 $EndComp
 $Comp
-L power:GND #PWR?
+L Data_Collection_KiCAD_Project-rescue:GND-power #PWR?
 U 1 1 616146B6
 P 2150 4350
@@
 NoConn ~ 2450 4150
 $Comp
-L power:+5V #PWR?
+L Data_Collection_KiCAD_Project-rescue:+5V-power #PWR?
 U 1 1 616146BE
 P 3300 3350
@@
 $EndComp
 $Comp
-L Power_Protection:USBLC6-2SC6 U?
+L Data_Collection_KiCAD_Project-rescue:USBLC6-2SC6-Power_Protection U?
 U 1 1 616146C5
 P 7400 4050
@@
 $EndComp
 $Comp
-L power:GND #PWR?
+L Data_Collection_KiCAD_Project-rescue:GND-power #PWR?
 U 1 1 616146CD
 P 7400 4450
@@
 $EndComp
 $Comp
-L power:+5V #PWR?
+L Data_Collection_KiCAD_Project-rescue:+5V-power #PWR?
 U 1 1 616146D7
 P 7400 3650
@@
 D-
 $Comp
-L Device:Ferrite_Bead_Small FB?
+L Data_Collection_KiCAD_Project-rescue:Ferrite_Bead_Small-Device FB?
 U 1 1 617A596A
 P 2800 3750
@@
 	5100 3900 5100 3750
 $Comp
-L Device:C C?
+L Data_Collection_KiCAD_Project-rescue:C-Device C?
 U 1 1 617B9DBE
 P 5100 4050
@@
 	3900 3900 3900 3750
 $Comp
-L Device:C C?
+L Data_Collection_KiCAD_Project-rescue:C-Device C?
 U 1 1 617B9DD7
 P 3900 4050
@@
 Connection ~ 5100 3750
 $Comp
-L Device:R R?
+L Data_Collection_KiCAD_Project-rescue:R-Device R?
 U 1 1 617B9DEE
 P 4750 3950
@@
 $EndComp
 $Comp
-L Device:R R?
+L Data_Collection_KiCAD_Project-rescue:R-Device R?
 U 1 1 617B9DF4
 P 4400 4350
@@
 LM317 Equation:\nVout = 1.25(1 + R2/R1)\nLet R1 = 240Ω, Vout = 3.3V\nR1 = 393.6Ω ≈ 390Ω
 $Comp
-L power:+3.3V #PWR?
+L Data_Collection_KiCAD_Project-rescue:+3.3V-power #PWR?
 U 1 1 617BD52E
 P 5100 2900
@@
 $EndComp
 $Comp
-L Device:LED D?
+L Data_Collection_KiCAD_Project-rescue:LED-Device D?
 U 1 1 617BEEA5
 P 5650 3750
@@
 $EndComp
 $Comp
-L Device:R R?
+L Data_Collection_KiCAD_Project-rescue:R-Device R?
 U 1 1 617BF66F
 P 6000 4150
@@
 	6000 3750 5800 3750
 $Comp
-L power:GND #PWR?
+L Data_Collection_KiCAD_Project-rescue:GND-power #PWR?
 U 1 1 617B9DC9
 P 4400 4500
@@
 $EndComp
 $Comp
-L power:GND #PWR?
+L Data_Collection_KiCAD_Project-rescue:GND-power #PWR?
 U 1 1 617C00BC
 P 3900 4200
@@
 $EndComp
 $Comp
-L power:GND #PWR?
+L Data_Collection_KiCAD_Project-rescue:GND-power #PWR?
 U 1 1 617C0723
 P 5100 4200
@@
 $EndComp
 $Comp
-L power:GND #PWR?
+L Data_Collection_KiCAD_Project-rescue:GND-power #PWR?
 U 1 1 617C0CB1
 P 6000 4300
@@
 USB shield to remain floating for USB Devices\nCan be connected to board enclosure if possible
 $Comp
-L Device:D_Zener D?
+L Data_Collection_KiCAD_Project-rescue:D_Zener-Device D?
 U 1 1 617F9817
 P 3500 3750
@@
 	3300 3750 2900 3750
 $Comp
-L Device:D_Zener D?
+L Data_Collection_KiCAD_Project-rescue:D_Zener-Device D?
 U 1 1 617FB0E6
 P 4400 3300
