File: Data_Collection_KiCAD_Project/file61A437B4.sch (KiCad schematic (older format))
At the start: 2 parts

Commit message: Corrected Main Bus Connector
Connections:
- net GND: now also C?.1; no longer C?.2
- net NRST: now also C?.2
- net at J?.13: no longer C?.1
Other:
- moved on the sheet: C?
Changed lines of the file:
@@
 Text HLabel 5250 2500 0    50   Input ~ 0
 SWCLK
-Text HLabel 5250 2600 0    50   Input ~ 0
+Text HLabel 4450 2600 0    50   Input ~ 0
 NRST
 $Comp
 L Device:C_Small C?
 U 1 1 61A55586
-P 5050 2700
+P 4450 2700
 AR Path="/61A55586" Ref="C?"  Part="1"
 AR Path="/61A437B5/61A55586" Ref="C?"  Part="1"
 AR Path="/619DD6DC/61A55586" Ref="C?"  Part="1"
-F 0 "C?" H 5142 2746 50  0000 L CNN
-F 1 "100nF" H 5142 2655 50  0000 L CNN
-F 2 "" H 5050 2700 50  0001 C CNN
-F 3 "~" H 5050 2700 50  0001 C CNN
-	1    5050 2700
-	0    1    1    0
+F 0 "C?" H 4550 2800 50  0000 L CNN
+F 1 "100nF" H 4550 2700 50  0000 L CNN
+F 2 "" H 4450 2700 50  0001 C CNN
+F 3 "~" H 4450 2700 50  0001 C CNN
+	1    4450 2700
+	-1   0    0    1
 $EndComp
-Wire Wire Line
-	5150 2700 5250 2700
 $Comp
 L power:GND #PWR?
 U 1 1 61A5558D
-P 4950 2700
+P 4450 2800
 AR Path="/61A5558D" Ref="#PWR?"  Part="1"
 AR Path="/61A437B5/61A5558D" Ref="#PWR?"  Part="1"
 AR Path="/619DD6DC/61A5558D" Ref="#PWR?"  Part="1"
-F 0 "#PWR?" H 4950 2450 50  0001 C CNN
-F 1 "GND" H 4955 2527 50  0000 C CNN
-F 2 "" H 4950 2700 50  0001 C CNN
-F 3 "" H 4950 2700 50  0001 C CNN
-	1    4950 2700
-	0    1    1    0
+F 0 "#PWR?" H 4450 2550 50  0001 C CNN
+F 1 "GND" H 4455 2627 50  0000 C CNN
+F 2 "" H 4450 2800 50  0001 C CNN
+F 3 "" H 4450 2800 50  0001 C CNN
+	1    4450 2800
+	1    0    0    -1
 $EndComp
 Text HLabel 5250 2800 0    50   Input ~ 0
@@
 Text HLabel 5250 2900 0    50   Input ~ 0
 Fire_redundant
+Wire Wire Line
+	4450 2600 5250 2600
 $EndSCHEMATC

Commit message: footprint changes
Parts:
- C24: renamed from C?; footprint (none) -> Capacitor_SMD:C_0603_1608Metric
- gave numbers to parts that had none: 1
Changed lines of the file:
@@
 $EndDescr
 $Comp
-L Connector:DB37_Male J?
+L Connector:DB37_Male J3
 U 1 1 61A44CBA
 P 5550 3300
-F 0 "J?" H 5730 3359 50  0000 L CNN
+F 0 "J3" H 5730 3359 50  0000 L CNN
 F 1 "DB37_Male" H 5730 3268 50  0000 L CNN
 F 2 "" H 5550 3300 50  0001 C CNN
@@
 $EndComp
 $Comp
-L power:Earth #PWR?
+L power:Earth #PWR053
 U 1 1 61A472F3
 P 5250 1500
-F 0 "#PWR?" H 5250 1250 50  0001 C CNN
+F 0 "#PWR053" H 5250 1250 50  0001 C CNN
 F 1 "Earth" H 5250 1350 50  0001 C CNN
 F 2 "" H 5250 1500 50  0001 C CNN
@@
 $EndComp
 $Comp
-L power:Earth #PWR?
+L power:Earth #PWR058
 U 1 1 61A486AF
 P 5250 5100
-F 0 "#PWR?" H 5250 4850 50  0001 C CNN
+F 0 "#PWR058" H 5250 4850 50  0001 C CNN
 F 1 "Earth" H 5250 4950 50  0001 C CNN
 F 2 "" H 5250 5100 50  0001 C CNN
@@
 $EndComp
 $Comp
-L power:+5V #PWR?
+L power:+5V #PWR054
 U 1 1 61A491E6
 P 5250 1600
-F 0 "#PWR?" H 5250 1450 50  0001 C CNN
+F 0 "#PWR054" H 5250 1450 50  0001 C CNN
 F 1 "+5V" V 5265 1728 50  0000 L CNN
 F 2 "" H 5250 1600 50  0001 C CNN
@@
 $EndComp
 $Comp
-L power:+5V #PWR?
+L power:+5V #PWR057
 U 1 1 61A49AB4
 P 5250 5000
-F 0 "#PWR?" H 5250 4850 50  0001 C CNN
+F 0 "#PWR057" H 5250 4850 50  0001 C CNN
 F 1 "+5V" V 5265 5128 50  0000 L CNN
 F 2 "" H 5250 5000 50  0001 C CNN
@@
 $EndComp
 $Comp
-L power:+3.3V #PWR?
+L power:+3.3V #PWR055
 U 1 1 61A4A3FB
 P 5250 1700
-F 0 "#PWR?" H 5250 1550 50  0001 C CNN
+F 0 "#PWR055" H 5250 1550 50  0001 C CNN
 F 1 "+3.3V" V 5265 1828 50  0000 L CNN
 F 2 "" H 5250 1700 50  0001 C CNN
@@
 $EndComp
 $Comp
-L power:+3.3V #PWR?
+L power:+3.3V #PWR056
 U 1 1 61A4AB5D
 P 5250 4900
-F 0 "#PWR?" H 5250 4750 50  0001 C CNN
+F 0 "#PWR056" H 5250 4750 50  0001 C CNN
 F 1 "+3.3V" V 5265 5028 50  0000 L CNN
 F 2 "" H 5250 4900 50  0001 C CNN
@@
 AR Path="/61A55586" Ref="C?"  Part="1"
 AR Path="/61A437B5/61A55586" Ref="C?"  Part="1"
-AR Path="/619DD6DC/61A55586" Ref="C?"  Part="1"
-F 0 "C?" H 4550 2800 50  0000 L CNN
+AR Path="/619DD6DC/61A55586" Ref="C24"  Part="1"
+F 0 "C24" H 4550 2800 50  0000 L CNN
 F 1 "100nF" H 4550 2700 50  0000 L CNN
-F 2 "" H 4450 2700 50  0001 C CNN
+F 2 "Capacitor_SMD:C_0603_1608Metric" H 4450 2700 50  0001 C CNN
 F 3 "~" H 4450 2700 50  0001 C CNN
 	1    4450 2700
@@
 AR Path="/61A5558D" Ref="#PWR?"  Part="1"
 AR Path="/61A437B5/61A5558D" Ref="#PWR?"  Part="1"
-AR Path="/619DD6DC/61A5558D" Ref="#PWR?"  Part="1"
-F 0 "#PWR?" H 4450 2550 50  0001 C CNN
+AR Path="/619DD6DC/61A5558D" Ref="#PWR052"  Part="1"
+F 0 "#PWR052" H 4450 2550 50  0001 C CNN
 F 1 "GND" H 4455 2627 50  0000 C CNN
 F 2 "" H 4450 2800 50  0001 C CNN
