File: Hardware/COMPONENT_SHEETS/MEMS_KX134.sch (KiCad schematic (older format))
At the start: 2 parts

Commit message: GPS layout change and test point tweaks
Parts:
- gave numbers to parts that had none: 2
Changed lines of the file:
@@
 $Descr A4 11693 8268
 encoding utf-8
-Sheet 8 10
+Sheet 5 10
 Title "ICM-20948 MEMS Chip"
 Date "2021-12-06"
@@
 $EndDescr
 $Comp
-L Data_Collection_KiCAD_Project-rescue:KX122-1042-Sensor_Motion-Data_Collection_KiCAD_Project-rescue U?
+L Data_Collection_KiCAD_Project-rescue:KX122-1042-Sensor_Motion-Data_Collection_KiCAD_Project-rescue U2
 U 1 1 6165C3D0
 P 5950 3450
-F 0 "U?" H 5950 4300 50  0000 C CNN
+F 0 "U2" H 5950 4300 50  0000 C CNN
 F 1 "KX134-1211" H 5950 4200 50  0000 C CNN
 F 2 "Package_LGA:LGA-12_2x2mm_P0.5mm" H 6100 4000 50  0001 L CNN
@@
 SCL
 $Comp
-L Data_Collection_KiCAD_Project-rescue:GND-power-Data_Collection_KiCAD_Project-rescue #PWR?
+L Data_Collection_KiCAD_Project-rescue:GND-power-Data_Collection_KiCAD_Project-rescue #PWR0107
 U 1 1 61692503
 P 5950 3950
-F 0 "#PWR?" H 5950 3700 50  0001 C CNN
+F 0 "#PWR0107" H 5950 3700 50  0001 C CNN
 F 1 "GND" H 5955 3777 50  0000 C CNN
 F 2 "" H 5950 3950 50  0001 C CNN
@@
 $EndComp
 $Comp
-L Data_Collection_KiCAD_Project-rescue:+3.3V-power-Data_Collection_KiCAD_Project-rescue #PWR?
+L Data_Collection_KiCAD_Project-rescue:+3.3V-power-Data_Collection_KiCAD_Project-rescue #PWR0108
 U 1 1 6169CC30
 P 5350 2900
-F 0 "#PWR?" H 5350 2750 50  0001 C CNN
+F 0 "#PWR0108" H 5350 2750 50  0001 C CNN
 F 1 "+3.3V" H 5365 3073 50  0000 C CNN
 F 2 "" H 5350 2900 50  0001 C CNN
@@
 $EndComp
 $Comp
-L Data_Collection_KiCAD_Project-rescue:C_Small-Device-Data_Collection_KiCAD_Project-rescue C?
+L Data_Collection_KiCAD_Project-rescue:C_Small-Device-Data_Collection_KiCAD_Project-rescue C23
 U 1 1 6169DA95
 P 6450 2900
-F 0 "C?" V 6221 2900 50  0000 C CNN
+F 0 "C23" V 6221 2900 50  0000 C CNN
 F 1 "0.1uF" V 6312 2900 50  0000 C CNN
 F 2 "Capacitor_SMD:C_0603_1608Metric" H 6450 2900 50  0001 C CNN
@@
 $EndComp
 $Comp
-L Data_Collection_KiCAD_Project-rescue:GND-power-Data_Collection_KiCAD_Project-rescue #PWR?
+L Data_Collection_KiCAD_Project-rescue:GND-power-Data_Collection_KiCAD_Project-rescue #PWR0109
 U 1 1 6169E39E
 P 6650 2900
-F 0 "#PWR?" H 6650 2650 50  0001 C CNN
+F 0 "#PWR0109" H 6650 2650 50  0001 C CNN
 F 1 "GND" H 6655 2727 50  0000 C CNN
 F 2 "" H 6650 2900 50  0001 C CNN
@@
 KX134-1211 I2C Addresses:\nADDR = 0 -> 0x1E\nADDR = 1 -> 0x1F
 $Comp
-L Data_Collection_KiCAD_Project-rescue:GND-power-Data_Collection_KiCAD_Project-rescue #PWR?
+L Data_Collection_KiCAD_Project-rescue:GND-power-Data_Collection_KiCAD_Project-rescue #PWR0110
 U 1 1 616ACA8D
 P 5200 3600
-F 0 "#PWR?" H 5200 3350 50  0001 C CNN
+F 0 "#PWR0110" H 5200 3350 50  0001 C CNN
 F 1 "GND" H 5205 3427 50  0000 C CNN
 F 2 "" H 5200 3600 50  0001 C CNN
@@
 	5200 3450 5200 3600
 $Comp
-L Data_Collection_KiCAD_Project-rescue:GND-power-Data_Collection_KiCAD_Project-rescue #PWR?
+L Data_Collection_KiCAD_Project-rescue:GND-power-Data_Collection_KiCAD_Project-rescue #PWR0111
 U 1 1 616AF0ED
 P 6700 3900
-F 0 "#PWR?" H 6700 3650 50  0001 C CNN
+F 0 "#PWR0111" H 6700 3650 50  0001 C CNN
 F 1 "GND" H 6705 3727 50  0000 C CNN
 F 2 "" H 6700 3900 50  0001 C CNN

Commit message: Schematic Tweaks and Board Dimensioned
Parts:
- C23: footprint Capacitor_SMD:C_0603_1608Metric -> Capacitor_SMD:C_0603_1608Metric_Pad1.08x0.95mm_HandSolder
Changed lines of the file:
@@
 F 0 "C23" V 6221 2900 50  0000 C CNN
 F 1 "0.1uF" V 6312 2900 50  0000 C CNN
-F 2 "Capacitor_SMD:C_0603_1608Metric" H 6450 2900 50  0001 C CNN
+F 2 "Capacitor_SMD:C_0603_1608Metric_Pad1.08x0.95mm_HandSolder" H 6450 2900 50  0001 C CNN
 F 3 "~" H 6450 2900 50  0001 C CNN
 	1    6450 2900
