File: Hardware/COMPONENT_SHEETS/DSUB.sch (KiCad schematic (older format))
At the start: 2 parts

Commit message: GPS layout change and test point tweaks
Parts:
- J3: renamed from J?; footprint L717SDC37P1ACH4F:L717SDC37P1ACH4F -> Connector_Dsub:DSUB-37_Male_Horizontal_P2.77x2.84mm_EdgePinOffset9.90mm_Housed_MountingHolesOffset11.32mm; symbol Charges_KiCAD_Project-rescue:L717SDC37P1ACH4F-SamacSys_Parts -> Data_Collection_KiCAD_Project-rescue:L717SDC37P1ACH4F-SamacSys_Parts-Charges_KiCAD_Project-rescue
Changed lines of the file:
@@
 	5300 2400 5700 2400
 $Comp
-L power:+3.3V #PWR?
+L power:+3.3V #PWR0122
 U 1 1 61A4A3FB
 P 6700 2000
-F 0 "#PWR?" H 6700 1850 50  0001 C CNN
+F 0 "#PWR0122" H 6700 1850 50  0001 C CNN
 F 1 "+3.3V" V 6715 2128 50  0000 L CNN
 F 2 "" H 6700 2000 50  0001 C CNN
@@
 $EndComp
 $Comp
-L power:+5V #PWR?
+L power:+5V #PWR0123
 U 1 1 61A491E6
 P 5700 1900
-F 0 "#PWR?" H 5700 1750 50  0001 C CNN
+F 0 "#PWR0123" H 5700 1750 50  0001 C CNN
 F 1 "+5V" V 5715 2028 50  0000 L CNN
 F 2 "" H 5700 1900 50  0001 C CNN
@@
 $EndComp
 $Comp
-L power:+3.3V #PWR?
+L power:+3.3V #PWR0124
 U 1 1 61A4AB5D
 P 6700 3600
-F 0 "#PWR?" H 6700 3450 50  0001 C CNN
+F 0 "#PWR0124" H 6700 3450 50  0001 C CNN
 F 1 "+3.3V" V 6715 3728 50  0000 L CNN
 F 2 "" H 6700 3600 50  0001 C CNN
@@
 $EndComp
 $Comp
-L power:GND #PWR?
+L power:GND #PWR0125
 U 1 1 61CFEBAB
 P 6200 1600
-F 0 "#PWR?" H 6200 1350 50  0001 C CNN
+F 0 "#PWR0125" H 6200 1350 50  0001 C CNN
 F 1 "GND" V 6200 1500 50  0000 R CNN
 F 2 "" H 6200 1600 50  0001 C CNN
@@
 $EndComp
 $Comp
-L Charges_KiCAD_Project-rescue:L717SDC37P1ACH4F-SamacSys_Parts J?
+L Data_Collection_KiCAD_Project-rescue:L717SDC37P1ACH4F-SamacSys_Parts-Charges_KiCAD_Project-rescue J?
 U 1 1 61D5E9EE
 P 6200 1600
-F 0 "J?" V 6019 1600 50  0000 C CNN
+AR Path="/61D5E9EE" Ref="J?"  Part="1"
+AR Path="/619DD6DC/61D5E9EE" Ref="J3"  Part="1"
+F 0 "J3" V 6019 1600 50  0000 C CNN
 F 1 "L717SDC37P1ACH4F" V 6110 1600 50  0000 C CNN
-F 2 "L717SDC37P1ACH4F:L717SDC37P1ACH4F" H 8450 1900 50  0001 L CNN
+F 2 "Connector_Dsub:DSUB-37_Male_Horizontal_P2.77x2.84mm_EdgePinOffset9.90mm_Housed_MountingHolesOffset11.32mm" H 8450 1900 50  0001 L CNN
 F 3 "https://cdn.amphenol-icc.com/media/wysiwyg/files/drawing/l717sdxxxp1ach4f.pdf" H 8450 1800 50  0001 L CNN
 F 4 "D-Sub Standard Connectors 37P Sz C Std Density Pin Screwlock 4-40" H 8450 1700 50  0001 L CNN "Description"
@@
 $EndComp
 $Comp
-L power:GND #PWR?
+L power:GND #PWR0126
 U 1 1 61D612F7
 P 6700 1900
-F 0 "#PWR?" H 6700 1650 50  0001 C CNN
+F 0 "#PWR0126" H 6700 1650 50  0001 C CNN
 F 1 "GND" V 6700 1800 50  0000 R CNN
 F 2 "" H 6700 1900 50  0001 C CNN
@@
 $EndComp
 $Comp
-L power:GND #PWR?
+L power:GND #PWR0127
 U 1 1 61CFE017
 P 6850 3700
-F 0 "#PWR?" H 6850 3450 50  0001 C CNN
+F 0 "#PWR0127" H 6850 3450 50  0001 C CNN
 F 1 "GND" H 6855 3527 50  0000 C CNN
 F 2 "" H 6850 3700 50  0001 C CNN
@@
 	6850 3700 6700 3700
 $Comp
-L power:GND #PWR?
+L power:GND #PWR0128
 U 1 1 61D6677B
 P 6200 4000
-F 0 "#PWR?" H 6200 3750 50  0001 C CNN
+F 0 "#PWR0128" H 6200 3750 50  0001 C CNN
 F 1 "GND" H 6205 3827 50  0000 C CNN
 F 2 "" H 6200 4000 50  0001 C CNN
@@
 $EndComp
 $Comp
-L power:+5V #PWR?
+L power:+5V #PWR0129
 U 1 1 61A49AB4
 P 5700 3600
-F 0 "#PWR?" H 5700 3450 50  0001 C CNN
+F 0 "#PWR0129" H 5700 3450 50  0001 C CNN
 F 1 "+5V" V 5715 3728 50  0000 L CNN
 F 2 "" H 5700 3600 50  0001 C CNN

Commit message: Finalized
Everything is routed. There are probably some things that need rerouting or adjustment.
Connections:
- net labels removed: +5V
- no-connect marks 0 -> 2
Other:
- note added: "I have disconnected the 5V DSUB from the Data Collection \nbecause I do not want a situation to arise where the small linear \nregulator is powering the other boards on the bus. 5V on this\n board is only for usb power."
Changed lines of the file:
@@
-$EndComp
-$Comp
-L power:+5V #PWR0123
-U 1 1 61A491E6
-P 5700 1900
-F 0 "#PWR0123" H 5700 1750 50  0001 C CNN
-F 1 "+5V" V 5715 2028 50  0000 L CNN
-F 2 "" H 5700 1900 50  0001 C CNN
-F 3 "" H 5700 1900 50  0001 C CNN
-	1    5700 1900
-	0    -1   1    0
 $EndComp
 $Comp
@@
 	1    0    0    -1
 $EndComp
-$Comp
-L power:+5V #PWR0129
-U 1 1 61A49AB4
-P 5700 3600
-F 0 "#PWR0129" H 5700 3450 50  0001 C CNN
-F 1 "+5V" V 5715 3728 50  0000 L CNN
-F 2 "" H 5700 3600 50  0001 C CNN
-F 3 "" H 5700 3600 50  0001 C CNN
-	1    5700 3600
-	0    -1   1    0
-$EndComp
+NoConn ~ 5700 1900
+NoConn ~ 5700 3600
+Text Notes 1600 2750 0    50   ~ 0
+I have disconnected the 5V DSUB from the Data Collection \nbecause I do not want a situation to arise where the small linear \nregulator is powering the other boards on the bus. 5V on this\n board is only for usb power.
 $EndSCHEMATC

Commit message: Schematic Tweaks and Board Dimensioned
Parts:
- added JP1: 5V Disconnect, Jumper:SolderJumper-2_P1.3mm_Bridged_Pad1.0x1.5mm, symbol Jumper:SolderJumper_2_Bridged
- C5: footprint Capacitor_SMD:C_0603_1608Metric -> Capacitor_SMD:C_0603_1608Metric_Pad1.08x0.95mm_HandSolder
Connections:
- net labels added: +5V, Dsub_5v
- wire segments 2 -> 4
- no-connect marks 2 -> 0
Changed lines of the file:
@@
 F 0 "C24" H 5292 2446 50  0000 L CNN
 F 1 "100nF" H 5292 2355 50  0000 L CNN
-F 2 "Capacitor_SMD:C_0603_1608Metric" H 5200 2400 50  0001 C CNN
+F 2 "Capacitor_SMD:C_0603_1608Metric_Pad1.08x0.95mm_HandSolder" H 5200 2400 50  0001 C CNN
 F 3 "~" H 5200 2400 50  0001 C CNN
 	1    5200 2400
@@
 $EndComp
 $Comp
-L Data_Collection_KiCAD_Project-rescue:L717SDC37P1ACH4F-SamacSys_Parts-Charges_KiCAD_Project-rescue J?
-U 1 1 61D5E9EE
-P 6200 1600
-AR Path="/61D5E9EE" Ref="J?"  Part="1"
-AR Path="/619DD6DC/61D5E9EE" Ref="J3"  Part="1"
-F 0 "J3" V 6019 1600 50  0000 C CNN
-F 1 "L717SDC37P1ACH4F" V 6110 1600 50  0000 C CNN
-F 2 "Connector_Dsub:DSUB-37_Male_Horizontal_P2.77x2.84mm_EdgePinOffset9.90mm_Housed_MountingHolesOffset11.32mm" H 8450 1900 50  0001 L CNN
-F 3 "https://cdn.amphenol-icc.com/media/wysiwyg/files/drawing/l717sdxxxp1ach4f.pdf" H 8450 1800 50  0001 L CNN
-F 4 "D-Sub Standard Connectors 37P Sz C Std Density Pin Screwlock 4-40" H 8450 1700 50  0001 L CNN "Description"
-F 5 "12.93" H 8450 1600 50  0001 L CNN "Height"
-F 6 "523-L717SDC37P1ACH4F" H 8450 1500 50  0001 L CNN "Mouser Part Number"
-F 7 "https://www.mouser.co.uk/ProductDetail/Amphenol-Commercial-Products/L717SDC37P1ACH4F?qs=wLKqLMNa9uLzTtnbxoO2Ng%3D%3D" H 8450 1400 50  0001 L CNN "Mouser Price/Stock"
-F 8 "Amphenol" H 8450 1300 50  0001 L CNN "Manufacturer_Name"
-F 9 "L717SDC37P1ACH4F" H 8450 1200 50  0001 L CNN "Manufacturer_Part_Number"
-	1    6200 1600
-	0    1    1    0
-$EndComp
-$Comp
 L power:GND #PWR0126
 U 1 1 61D612F7
@@
 	1    0    0    -1
 $EndComp
-NoConn ~ 5700 1900
-NoConn ~ 5700 3600
 Text Notes 1600 2750 0    50   ~ 0
 I have disconnected the 5V DSUB from the Data Collection \nbecause I do not want a situation to arise where the small linear \nregulator is powering the other boards on the bus. 5V on this\n board is only for usb power.
+Text Label 5700 1900 2    50   ~ 0
+Dsub_5v
+$Comp
+L Data_Collection_KiCAD_Project-rescue:L717SDC37P1ACH4F-SamacSys_Parts-Charges_KiCAD_Project-rescue J?
+U 1 1 61D5E9EE
+P 6200 1600
+AR Path="/61D5E9EE" Ref="J?"  Part="1"
+AR Path="/619DD6DC/61D5E9EE" Ref="J3"  Part="1"
+F 0 "J3" V 6019 1600 50  0000 C CNN
+F 1 "L717SDC37P1ACH4F" V 6110 1600 50  0000 C CNN
+F 2 "Connector_Dsub:DSUB-37_Male_Horizontal_P2.77x2.84mm_EdgePinOffset9.90mm_Housed_MountingHolesOffset11.32mm" H 8450 1900 50  0001 L CNN
+F 3 "https://cdn.amphenol-icc.com/media/wysiwyg/files/drawing/l717sdxxxp1ach4f.pdf" H 8450 1800 50  0001 L CNN
+F 4 "D-Sub Standard Connectors 37P Sz C Std Density Pin Screwlock 4-40" H 8450 1700 50  0001 L CNN "Description"
+F 5 "12.93" H 8450 1600 50  0001 L CNN "Height"
+F 6 "523-L717SDC37P1ACH4F" H 8450 1500 50  0001 L CNN "Mouser Part Number"
+F 7 "https://www.mouser.co.uk/ProductDetail/Amphenol-Commercial-Products/L717SDC37P1ACH4F?qs=wLKqLMNa9uLzTtnbxoO2Ng%3D%3D" H 8450 1400 50  0001 L CNN "Mouser Price/Stock"
+F 8 "Amphenol" H 8450 1300 50  0001 L CNN "Manufacturer_Name"
+F 9 "L717SDC37P1ACH4F" H 8450 1200 50  0001 L CNN "Manufacturer_Part_Number"
+	1    6200 1600
+	0    1    1    0
+$EndComp
+Text Label 5700 3600 2    50   ~ 0
+Dsub_5v
+$Comp
+L Jumper:SolderJumper_2_Bridged JP1
+U 1 1 61C3ADEE
+P 2750 3200
+F 0 "JP1" H 2750 3405 50  0000 C CNN
+F 1 "5V Disconnect" H 2750 3314 50  0000 C CNN
+F 2 "Jumper:SolderJumper-2_P1.3mm_Bridged_Pad1.0x1.5mm" H 2750 3200 50  0001 C CNN
+F 3 "~" H 2750 3200 50  0001 C CNN
+	1    2750 3200
+	1    0    0    -1
+$EndComp
+Text Label 3100 3200 0    50   ~ 0
+Dsub_5v
+$Comp
+L power:+5V #PWR0123
+U 1 1 61C3CDC8
+P 2150 3200
+F 0 "#PWR0123" H 2150 3050 50  0001 C CNN
+F 1 "+5V" H 2165 3373 50  0000 C CNN
+F 2 "" H 2150 3200 50  0001 C CNN
+F 3 "" H 2150 3200 50  0001 C CNN
+	1    2150 3200
+	1    0    0    -1
+$EndComp
+Wire Wire Line
+	2600 3200 2150 3200
+Wire Wire Line
+	2900 3200 3100 3200
 $EndSCHEMATC

Commit message: routing progress and pin reassignment
Parts:
- J3: footprint Connector_Dsub:DSUB-37_Male_Horizontal_P2.77x2.84mm_EdgePinOffset9.90mm_Housed_MountingHolesOffset11.32mm -> RDT_Custom_Footprints:L717SDC37P1ACH4F
Changed lines of the file:
@@
 F 0 "J3" V 6019 1600 50  0000 C CNN
 F 1 "L717SDC37P1ACH4F" V 6110 1600 50  0000 C CNN
-F 2 "Connector_Dsub:DSUB-37_Male_Horizontal_P2.77x2.84mm_EdgePinOffset9.90mm_Housed_MountingHolesOffset11.32mm" H 8450 1900 50  0001 L CNN
+F 2 "RDT_Custom_Footprints:L717SDC37P1ACH4F" H 8450 1900 50  0001 L CNN
 F 3 "https://cdn.amphenol-icc.com/media/wysiwyg/files/drawing/l717sdxxxp1ach4f.pdf" H 8450 1800 50  0001 L CNN
 F 4 "D-Sub Standard Connectors 37P Sz C Std Density Pin Screwlock 4-40" H 8450 1700 50  0001 L CNN "Description"
