File: Hardware/COMPONENT_SHEETS/USB_ESD.sch (KiCad schematic (older format))
At the start: 9 parts, among them U1 LM317T

Commit message: GPS layout change and test point tweaks
Parts:
- gave numbers to parts that had none: 4
Changed lines of the file:
@@
 $Descr A4 11693 8268
 encoding utf-8
-Sheet 2 10
+Sheet 8 10
 Title "USB Connector and ESD Protection"
 Date "2021-12-06"
@@
 $EndDescr
 $Comp
-L Data_Collection_KiCAD_Project-rescue:USB_B_Micro-Connector-Data_Collection_KiCAD_Project-rescue J?
+L Data_Collection_KiCAD_Project-rescue:USB_B_Micro-Connector-Data_Collection_KiCAD_Project-rescue J1
 U 1 1 616146B0
 P 2150 3950
-F 0 "J?" H 2300 4300 50  0000 C CNN
+F 0 "J1" H 2300 4300 50  0000 C CNN
 F 1 "USB_B_Micro" H 2450 3600 50  0000 C CNN
 F 2 "Connector_USB:USB_Micro-B_Amphenol_10103594-0001LF_Horizontal" H 2300 3900 50  0001 C CNN
@@
 $EndComp
 $Comp
-L Data_Collection_KiCAD_Project-rescue:GND-power-Data_Collection_KiCAD_Project-rescue #PWR?
+L Data_Collection_KiCAD_Project-rescue:GND-power-Data_Collection_KiCAD_Project-rescue #PWR0112
 U 1 1 616146B6
 P 2150 4350
-F 0 "#PWR?" H 2150 4100 50  0001 C CNN
+F 0 "#PWR0112" H 2150 4100 50  0001 C CNN
 F 1 "GND" H 2155 4177 50  0000 C CNN
 F 2 "" H 2150 4350 50  0001 C CNN
@@
 NoConn ~ 2450 4150
 $Comp
-L Data_Collection_KiCAD_Project-rescue:+5V-power-Data_Collection_KiCAD_Project-rescue #PWR?
+L Data_Collection_KiCAD_Project-rescue:+5V-power-Data_Collection_KiCAD_Project-rescue #PWR0113
 U 1 1 616146BE
 P 3650 3350
-F 0 "#PWR?" H 3650 3200 50  0001 C CNN
+F 0 "#PWR0113" H 3650 3200 50  0001 C CNN
 F 1 "+5V" H 3665 3523 50  0000 C CNN
 F 2 "" H 3650 3350 50  0001 C CNN
@@
 $EndComp
 $Comp
-L Data_Collection_KiCAD_Project-rescue:USBLC6-2SC6-Power_Protection-Data_Collection_KiCAD_Project-rescue U?
+L Data_Collection_KiCAD_Project-rescue:USBLC6-2SC6-Power_Protection-Data_Collection_KiCAD_Project-rescue U5
 U 1 1 616146C5
 P 7400 4050
-F 0 "U?" H 7650 4400 50  0000 C CNN
+F 0 "U5" H 7650 4400 50  0000 C CNN
 F 1 "USBLC6-2SC6" H 7700 3700 50  0000 C CNN
 F 2 "Package_TO_SOT_SMD:SOT-23-6" H 7400 3550 50  0001 C CNN
@@
 $EndComp
 $Comp
-L Data_Collection_KiCAD_Project-rescue:GND-power-Data_Collection_KiCAD_Project-rescue #PWR?
+L Data_Collection_KiCAD_Project-rescue:GND-power-Data_Collection_KiCAD_Project-rescue #PWR0114
 U 1 1 616146CD
 P 7400 4450
-F 0 "#PWR?" H 7400 4200 50  0001 C CNN
+F 0 "#PWR0114" H 7400 4200 50  0001 C CNN
 F 1 "GND" H 7405 4277 50  0000 C CNN
 F 2 "" H 7400 4450 50  0001 C CNN
@@
 $EndComp
 $Comp
-L Data_Collection_KiCAD_Project-rescue:+5V-power-Data_Collection_KiCAD_Project-rescue #PWR?
+L Data_Collection_KiCAD_Project-rescue:+5V-power-Data_Collection_KiCAD_Project-rescue #PWR0115
 U 1 1 616146D7
 P 7400 3650
-F 0 "#PWR?" H 7400 3500 50  0001 C CNN
+F 0 "#PWR0115" H 7400 3500 50  0001 C CNN
 F 1 "+5V" H 7415 3823 50  0000 C CNN
 F 2 "" H 7400 3650 50  0001 C CNN
@@
 D-
 $Comp
-L Data_Collection_KiCAD_Project-rescue:Ferrite_Bead_Small-Device-Data_Collection_KiCAD_Project-rescue FB?
+L Data_Collection_KiCAD_Project-rescue:Ferrite_Bead_Small-Device-Data_Collection_KiCAD_Project-rescue FB1
 U 1 1 617A596A
 P 2800 3750
-F 0 "FB?" V 2563 3750 50  0000 C CNN
+F 0 "FB1" V 2563 3750 50  0000 C CNN
 F 1 "Ferrite_Bead_Small" V 2654 3750 50  0000 C CNN
 F 2 "Capacitor_SMD:C_0603_1608Metric" V 2730 3750 50  0001 C CNN
@@
 AR Path="/615A5159/617B9DBE" Ref="C?"  Part="1"
 AR Path="/615EE01A/617B9DBE" Ref="C2"  Part="1"
-F 0 "C?" H 5215 4096 50  0000 L CNN
+F 0 "C2" H 5215 4096 50  0000 L CNN
 F 1 "1uF" H 5215 4005 50  0000 L CNN
 F 2 "Capacitor_SMD:C_0603_1608Metric" H 5138 3900 50  0001 C CNN
@@
 AR Path="/615A5159/617B9DD7" Ref="C?"  Part="1"
 AR Path="/615EE01A/617B9DD7" Ref="C1"  Part="1"
-F 0 "C?" H 4015 4096 50  0000 L CNN
+F 0 "C1" H 4015 4096 50  0000 L CNN
 F 1 "0.1uF" H 4015 4005 50  0000 L CNN
 F 2 "Capacitor_SMD:C_0603_1608Metric" H 3938 3900 50  0001 C CNN
@@
 AR Path="/615A5159/617B9DE6" Ref="U?"  Part="1"
 AR Path="/615EE01A/617B9DE6" Ref="U1"  Part="1"
-F 0 "U?" H 4400 4037 60  0000 C CNN
+F 0 "U1" H 4400 4037 60  0000 C CNN
 F 1 "LM317T" H 4400 3931 60  0000 C CNN
 F 2 "digikey-footprints:TO-220-3" H 4600 3950 60  0001 L CNN
@@
 AR Path="/615A5159/617B9DEE" Ref="R?"  Part="1"
 AR Path="/615EE01A/617B9DEE" Ref="R2"  Part="1"
-F 0 "R?" H 4820 3996 50  0000 L CNN
+F 0 "R2" H 4820 3996 50  0000 L CNN
 F 1 "240" H 4820 3905 50  0000 L CNN
 F 2 "Resistor_SMD:R_0603_1608Metric" V 4680 3950 50  0001 C CNN
@@
 AR Path="/615A5159/617B9DF4" Ref="R?"  Part="1"
 AR Path="/615EE01A/617B9DF4" Ref="R1"  Part="1"
-F 0 "R?" H 4470 4396 50  0000 L CNN
+F 0 "R1" H 4470 4396 50  0000 L CNN
 F 1 "390" H 4470 4305 50  0000 L CNN
 F 2 "Resistor_SMD:R_0603_1608Metric" V 4330 4350 50  0001 C CNN
@@
 AR Path="/617BD52E" Ref="#PWR?"  Part="1"
 AR Path="/615EE01A/617BD52E" Ref="#PWR09"  Part="1"
-F 0 "#PWR?" H 5100 2750 50  0001 C CNN
+F 0 "#PWR09" H 5100 2750 50  0001 C CNN
 F 1 "+3.3V" H 5115 3073 50  0000 C CNN
 F 2 "" H 5100 2900 50  0001 C CNN
@@
 AR Path="/615A5159/617B9DC9" Ref="#PWR?"  Part="1"
 AR Path="/615EE01A/617B9DC9" Ref="#PWR08"  Part="1"
-F 0 "#PWR?" H 4400 4250 50  0001 C CNN
+F 0 "#PWR08" H 4400 4250 50  0001 C CNN
 F 1 "GND" H 4405 4327 50  0000 C CNN
 F 2 "" H 4400 4500 50  0001 C CNN
@@
 AR Path="/615A5159/617C00BC" Ref="#PWR?"  Part="1"
 AR Path="/615EE01A/617C00BC" Ref="#PWR07"  Part="1"
-F 0 "#PWR?" H 3900 3950 50  0001 C CNN
+F 0 "#PWR07" H 3900 3950 50  0001 C CNN
 F 1 "GND" H 3905 4027 50  0000 C CNN
 F 2 "" H 3900 4200 50  0001 C CNN
@@
 AR Path="/615A5159/617C0723" Ref="#PWR?"  Part="1"
 AR Path="/615EE01A/617C0723" Ref="#PWR010"  Part="1"
-F 0 "#PWR?" H 5100 3950 50  0001 C CNN
+F 0 "#PWR010" H 5100 3950 50  0001 C CNN
 F 1 "GND" H 5105 4027 50  0000 C CNN
 F 2 "" H 5100 4200 50  0001 C CNN
@@
 Connection ~ 3900 3750
 $Comp
-L Device:D_Schottky D?
+L Device:D_Schottky D1
 U 1 1 61B1913C
 P 3400 3750
-F 0 "D?" H 3400 3533 50  0000 C CNN
+F 0 "D1" H 3400 3533 50  0000 C CNN
 F 1 "D_Schottky" H 3400 3624 50  0000 C CNN
 F 2 "Diode_SMD:D_0603_1608Metric" H 3400 3750 50  0001 C CNN

Commit message: Schematic Tweaks and Board Dimensioned
Parts:
- removed J1: USB_B_Micro, Connector_USB:USB_Micro-B_Amphenol_10103594-0001LF_Horizontal, symbol Data_Collection_KiCAD_Project-rescue:USB_B_Micro-Connector-Data_Collection_KiCA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
- added J1: 10118192-0001LF, Connector_USB:USB_Micro-B_Wuerth_614105150721_Vertical, symbol dk_USB-DVI-HDMI-Connectors:10118192-0001LF
- C1, C2, FB1: footprint Capacitor_SMD:C_0603_1608Metric -> Capacitor_SMD:C_0603_1608Metric_Pad1.08x0.95mm_HandSolder
- D1: footprint Diode_SMD:D_0603_1608Metric -> Diode_SMD:D_0603_1608Metric_Pad1.05x0.95mm_HandSolder
- R1, R2: footprint Resistor_SMD:R_0603_1608Metric -> Resistor_SMD:R_0603_1608Metric_Pad0.98x0.95mm_HandSolder
Connections:
- wire segments 16 -> 18
Changed lines of the file:
@@
 $EndDescr
-$Comp
-L Data_Collection_KiCAD_Project-rescue:USB_B_Micro-Connector-Data_Collection_KiCAD_Project-rescue J1
-U 1 1 616146B0
-P 2150 3950
-F 0 "J1" H 2300 4300 50  0000 C CNN
-F 1 "USB_B_Micro" H 2450 3600 50  0000 C CNN
-F 2 "Connector_USB:USB_Micro-B_Amphenol_10103594-0001LF_Horizontal" H 2300 3900 50  0001 C CNN
-F 3 "~" H 2300 3900 50  0001 C CNN
-	1    2150 3950
-	1    0    0    -1
-$EndComp
 $Comp
 L Data_Collection_KiCAD_Project-rescue:GND-power-Data_Collection_KiCAD_Project-rescue #PWR0112
 U 1 1 616146B6
-P 2150 4350
-F 0 "#PWR0112" H 2150 4100 50  0001 C CNN
-F 1 "GND" H 2155 4177 50  0000 C CNN
-F 2 "" H 2150 4350 50  0001 C CNN
-F 3 "" H 2150 4350 50  0001 C CNN
-	1    2150 4350
-	1    0    0    -1
-$EndComp
-NoConn ~ 2050 4350
-NoConn ~ 2450 4150
+P 2400 4300
+F 0 "#PWR0112" H 2400 4050 50  0001 C CNN
+F 1 "GND" H 2405 4127 50  0000 C CNN
+F 2 "" H 2400 4300 50  0001 C CNN
+F 3 "" H 2400 4300 50  0001 C CNN
+	1    2400 4300
+	1    0    0    -1
+$EndComp
+NoConn ~ 2300 4050
 $Comp
 L Data_Collection_KiCAD_Project-rescue:+5V-power-Data_Collection_KiCAD_Project-rescue #PWR0113
@@
 	1    0    0    -1
 $EndComp
-Text Notes 2950 3350 2    100  ~ 0
+Text Notes 2900 2750 2    100  ~ 0
 USB Connector
 Text HLabel 7000 3950 0    50   Input ~ 0
@@
 Text HLabel 7800 3950 2    50   Input ~ 0
 USB_CONN_D-
-Text HLabel 2450 3950 2    50   Output ~ 0
+Text HLabel 2300 3950 2    50   Output ~ 0
 USB_CONN_D+
-Text HLabel 2450 4050 2    50   Output ~ 0
+Text HLabel 2300 3850 2    50   Output ~ 0
 USB_CONN_D-
 Text HLabel 7000 4150 0    50   Output ~ 0
@@
 F 0 "FB1" V 2563 3750 50  0000 C CNN
 F 1 "Ferrite_Bead_Small" V 2654 3750 50  0000 C CNN
-F 2 "Capacitor_SMD:C_0603_1608Metric" V 2730 3750 50  0001 C CNN
+F 2 "Capacitor_SMD:C_0603_1608Metric_Pad1.08x0.95mm_HandSolder" V 2730 3750 50  0001 C CNN
 F 3 "~" H 2800 3750 50  0001 C CNN
 	1    2800 3750
 	0    1    1    0
 $EndComp
-Wire Wire Line
-	2700 3750 2450 3750
 Wire Notes Line
 	3750 4950 5400 4950
@@
 F 0 "C2" H 5215 4096 50  0000 L CNN
 F 1 "1uF" H 5215 4005 50  0000 L CNN
-F 2 "Capacitor_SMD:C_0603_1608Metric" H 5138 3900 50  0001 C CNN
+F 2 "Capacitor_SMD:C_0603_1608Metric_Pad1.08x0.95mm_HandSolder" H 5138 3900 50  0001 C CNN
 F 3 "~" H 5100 4050 50  0001 C CNN
 	1    5100 4050
@@
 F 0 "C1" H 4015 4096 50  0000 L CNN
 F 1 "0.1uF" H 4015 4005 50  0000 L CNN
-F 2 "Capacitor_SMD:C_0603_1608Metric" H 3938 3900 50  0001 C CNN
+F 2 "Capacitor_SMD:C_0603_1608Metric_Pad1.08x0.95mm_HandSolder" H 3938 3900 50  0001 C CNN
 F 3 "~" H 3900 4050 50  0001 C CNN
 	1    3900 4050
@@
 F 0 "R2" H 4820 3996 50  0000 L CNN
 F 1 "240" H 4820 3905 50  0000 L CNN
-F 2 "Resistor_SMD:R_0603_1608Metric" V 4680 3950 50  0001 C CNN
+F 2 "Resistor_SMD:R_0603_1608Metric_Pad0.98x0.95mm_HandSolder" V 4680 3950 50  0001 C CNN
 F 3 "~" H 4750 3950 50  0001 C CNN
 	1    4750 3950
@@
 F 0 "R1" H 4470 4396 50  0000 L CNN
 F 1 "390" H 4470 4305 50  0000 L CNN
-F 2 "Resistor_SMD:R_0603_1608Metric" V 4330 4350 50  0001 C CNN
+F 2 "Resistor_SMD:R_0603_1608Metric_Pad0.98x0.95mm_HandSolder" V 4330 4350 50  0001 C CNN
 F 3 "~" H 4400 4350 50  0001 C CNN
 	1    4400 4350
@@
 Wire Notes Line
 	6300 3400 6300 4700
-Wire Notes Line
-	3200 4650 3200 3400
-Wire Notes Line
-	3200 3400 1850 3400
-Wire Notes Line
-	1850 3400 1850 4650
-Wire Notes Line
-	1850 4650 3200 4650
 Text Notes 1600 4850 0    50   ~ 0
 USB shield to remain floating for USB Devices\nCan be connected to board enclosure if possible
@@
 F 0 "D1" H 3400 3533 50  0000 C CNN
 F 1 "D_Schottky" H 3400 3624 50  0000 C CNN
-F 2 "Diode_SMD:D_0603_1608Metric" H 3400 3750 50  0001 C CNN
+F 2 "Diode_SMD:D_0603_1608Metric_Pad1.05x0.95mm_HandSolder" H 3400 3750 50  0001 C CNN
 F 3 "~" H 3400 3750 50  0001 C CNN
 	1    3400 3750
@@
 	3550 3750 3650 3750
 Connection ~ 3650 3750
+$Comp
+L dk_USB-DVI-HDMI-Connectors:10118192-0001LF J1
+U 1 1 61C12C59
+P 2000 3950
+F 0 "J1" H 2064 4695 60  0000 C CNN
+F 1 "10118192-0001LF" H 2064 4589 60  0000 C CNN
+F 2 "Connector_USB:USB_Micro-B_Wuerth_614105150721_Vertical" H 2200 4150 60  0001 L CNN
+F 3 "http://www.amphenol-icc.com/media/wysiwyg/files/drawing/10118192.pdf" H 2200 4250 60  0001 L CNN
+F 4 "609-4613-1-ND" H 2200 4350 60  0001 L CNN "Digi-Key_PN"
+F 5 "10118192-0001LF" H 2200 4450 60  0001 L CNN "MPN"
+F 6 "Connectors, Interconnects" H 2200 4550 60  0001 L CNN "Category"
+F 7 "USB, DVI, HDMI Connectors" H 2200 4650 60  0001 L CNN "Family"
+F 8 "http://www.amphenol-icc.com/media/wysiwyg/files/drawing/10118192.pdf" H 2200 4750 60  0001 L CNN "DK_Datasheet_Link"
+F 9 "/product-detail/en/amphenol-icc-fci/10118192-0001LF/609-4613-1-ND/2785378" H 2200 4850 60  0001 L CNN "DK_Detail_Page"
+F 10 "CONN RCPT USB2.0 MICRO B SMD R/A" H 2200 4950 60  0001 L CNN "Description"
+F 11 "Amphenol ICC (FCI)" H 2200 5050 60  0001 L CNN "Manufacturer"
+F 12 "Active" H 2200 5150 60  0001 L CNN "Status"
+	1    2000 3950
+	1    0    0    -1
+$EndComp
+Wire Wire Line
+	2300 3750 2700 3750
+Wire Wire Line
+	2400 4300 2400 4150
+Wire Wire Line
+	2400 4150 2300 4150
+NoConn ~ 1900 4550
 $EndSCHEMATC

Commit message: routing progress and pin reassignment
Connections:
- no-connect marks 2 -> 1
Changed lines of the file:
@@
 Wire Wire Line
 	2400 4150 2300 4150
-NoConn ~ 1900 4550
 $EndSCHEMATC
