File: Hardware/COMPONENT_SHEETS/BAROMETER_MS5607-02.sch (KiCad schematic (older format))
At the start: 2 parts, among them U7 MS5607-02BA

Commit message: Schematic Tweaks and Board Dimensioned
Parts:
- C18: footprint Capacitor_SMD:C_0603_1608Metric -> Capacitor_SMD:C_0603_1608Metric_Pad1.08x0.95mm_HandSolder
Changed lines of the file:
@@
 F 0 "C18" H 6465 3696 50  0000 L CNN
 F 1 "100nF" H 6465 3605 50  0000 L CNN
-F 2 "Capacitor_SMD:C_0603_1608Metric" H 6388 3500 50  0001 C CNN
+F 2 "Capacitor_SMD:C_0603_1608Metric_Pad1.08x0.95mm_HandSolder" H 6388 3500 50  0001 C CNN
 F 3 "~" H 6350 3650 50  0001 C CNN
 	1    6350 3650
