File: Hardware/COMPONENT_SHEETS/FLASH_W25Q32JV.sch (KiCad schematic (older format))
At the start: 2 parts, among them U6 W25Q32JVSS

Commit message: Schematic Tweaks and Board Dimensioned
Parts:
- C17: footprint Capacitor_SMD:C_0603_1608Metric -> Capacitor_SMD:C_0603_1608Metric_Pad1.08x0.95mm_HandSolder
Changed lines of the file:
@@
 F 0 "C17" H 3965 3196 50  0000 L CNN
 F 1 "100nF" H 3965 3105 50  0000 L CNN
-F 2 "Capacitor_SMD:C_0603_1608Metric" H 3888 3000 50  0001 C CNN
+F 2 "Capacitor_SMD:C_0603_1608Metric_Pad1.08x0.95mm_HandSolder" H 3888 3000 50  0001 C CNN
 F 3 "~" H 3850 3150 50  0001 C CNN
 	1    3850 3150

Commit message: finished routing
Parts:
- removed C17: 100nF, Capacitor_SMD:C_0603_1608Metric_Pad1.08x0.95mm_HandSolder, symbol Data_Collection_KiCAD_Project-rescue:C-Device-Data_Collection_KiCAD_Project-res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
Changed lines of the file:
@@
 Text Notes 5150 2250 2    100  ~ 0
 Flash Storage Chip
-$Comp
-L Data_Collection_KiCAD_Project-rescue:C-Device-Data_Collection_KiCAD_Project-rescue C?
-U 1 1 6161186E
-P 3850 3150
-AR Path="/6161186E" Ref="C?"  Part="1"
-AR Path="/615FC266/6161186E" Ref="C17"  Part="1"
-F 0 "C17" H 3965 3196 50  0000 L CNN
-F 1 "100nF" H 3965 3105 50  0000 L CNN
-F 2 "Capacitor_SMD:C_0603_1608Metric_Pad1.08x0.95mm_HandSolder" H 3888 3000 50  0001 C CNN
-F 3 "~" H 3850 3150 50  0001 C CNN
-	1    3850 3150
-	1    0    0    -1
-$EndComp
 Text HLabel 4450 3300 0    50   Input ~ 0
 CLK
@@
 	5500 3450 5500 3400
 Connection ~ 5500 3400
-$Comp
-L Data_Collection_KiCAD_Project-rescue:GND-power-Data_Collection_KiCAD_Project-rescue #PWR?
-U 1 1 617DFAF5
-P 3850 3300
-AR Path="/617DFAF5" Ref="#PWR?"  Part="1"
-AR Path="/615FC266/617DFAF5" Ref="#PWR035"  Part="1"
-F 0 "#PWR035" H 3850 3050 50  0001 C CNN
-F 1 "GND" H 3855 3127 50  0000 C CNN
-F 2 "" H 3850 3300 50  0001 C CNN
-F 3 "" H 3850 3300 50  0001 C CNN
-	1    3850 3300
-	1    0    0    -1
-$EndComp
 Wire Wire Line
 	3850 3000 3850 2750
