File: Hardware/COMPONENT_SHEETS/GNSS_MAX-8Q.sch (KiCad schematic (older format))
At the start: 13 parts, among them J2 Conn_Coaxial, Q1 SI1040X-T1-GE3, U4 MAX-8Q

Commit message: GPS layout change and test point tweaks
Parts:
- L1: footprint Inductor_THT:L_Radial_D10.5mm_P5.00mm_Abacron_AISR-01 -> Inductor_SMD:L_0603_1608Metric; Digikey https://www.digikey.com/en/products/detail/abracon-llc/AIUR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 -> https://www.digikey.com/en/products/detail/murata-electroni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; Field5 (none) -> LQG15HS27NJ02
Changed lines of the file:
@@
 $Descr A4 11693 8268
 encoding utf-8
-Sheet 4 10
+Sheet 7 10
 Title "MAX-8Q GNSS Module"
 Date "2021-12-06"
@@
 AR Path="/616192D6" Ref="#PWR?"  Part="1"
 AR Path="/615A5F2C/616192D6" Ref="#PWR018"  Part="1"
-F 0 "#PWR?" H 4000 6250 50  0001 C CNN
+F 0 "#PWR018" H 4000 6250 50  0001 C CNN
 F 1 "GND" H 4005 6327 50  0000 C CNN
 F 2 "" H 4000 6500 50  0001 C CNN
@@
 AR Path="/616192DC" Ref="C?"  Part="1"
 AR Path="/615A5F2C/616192DC" Ref="C9"  Part="1"
-F 0 "C?" H 5015 5596 50  0000 L CNN
+F 0 "C9" H 5015 5596 50  0000 L CNN
 F 1 "1nF" H 5015 5505 50  0000 L CNN
 F 2 "Capacitor_SMD:C_0603_1608Metric" H 4938 5400 50  0001 C CNN
@@
 AR Path="/616192E2" Ref="R?"  Part="1"
 AR Path="/615A5F2C/616192E2" Ref="R5"  Part="1"
-F 0 "R?" H 4770 5596 50  0000 L CNN
+F 0 "R5" H 4770 5596 50  0000 L CNN
 F 1 "100k" H 4770 5505 50  0000 L CNN
 F 2 "Resistor_SMD:R_0603_1608Metric" V 4630 5550 50  0001 C CNN
@@
 AR Path="/616192E8" Ref="R?"  Part="1"
 AR Path="/615A5F2C/616192E8" Ref="R4"  Part="1"
-F 0 "R?" H 4420 6296 50  0000 L CNN
+F 0 "R4" H 4420 6296 50  0000 L CNN
 F 1 "10k" H 4420 6205 50  0000 L CNN
 F 2 "Resistor_SMD:R_0603_1608Metric" V 4280 6250 50  0001 C CNN
@@
 AR Path="/616192FE" Ref="#PWR?"  Part="1"
 AR Path="/615A5F2C/616192FE" Ref="#PWR019"  Part="1"
-F 0 "#PWR?" H 4900 5500 50  0001 C CNN
+F 0 "#PWR019" H 4900 5500 50  0001 C CNN
 F 1 "GND" H 4905 5577 50  0000 C CNN
 F 2 "" H 4900 5750 50  0001 C CNN
@@
 AR Path="/6161C95B" Ref="#PWR?"  Part="1"
 AR Path="/615A5F2C/6161C95B" Ref="#PWR021"  Part="1"
-F 0 "#PWR?" H 7200 2250 50  0001 C CNN
+F 0 "#PWR021" H 7200 2250 50  0001 C CNN
 F 1 "+3.3V" H 7215 2573 50  0000 C CNN
 F 2 "" H 7200 2400 50  0001 C CNN
@@
 AR Path="/6161C967" Ref="#PWR?"  Part="1"
 AR Path="/615A5F2C/6161C967" Ref="#PWR022"  Part="1"
-F 0 "#PWR?" H 7700 3650 50  0001 C CNN
+F 0 "#PWR022" H 7700 3650 50  0001 C CNN
 F 1 "GND" H 7705 3727 50  0000 C CNN
 F 2 "" H 7700 3900 50  0001 C CNN
@@
 AR Path="/6161C976" Ref="J?"  Part="1"
 AR Path="/615A5F2C/6161C976" Ref="J2"  Part="1"
-F 0 "J?" H 9500 3175 50  0000 L CNN
+F 0 "J2" H 9500 3175 50  0000 L CNN
 F 1 "Conn_Coaxial" H 9500 3084 50  0000 L CNN
 F 2 "Connector_Coaxial:SMA_Amphenol_132134-11_Vertical" H 9400 3200 50  0001 C CNN
@@
 AR Path="/6161C998" Ref="#PWR?"  Part="1"
 AR Path="/615A5F2C/6161C998" Ref="#PWR017"  Part="1"
-F 0 "#PWR?" H 1200 1700 50  0001 C CNN
+F 0 "#PWR017" H 1200 1700 50  0001 C CNN
 F 1 "GND" H 1205 1777 50  0000 C CNN
 F 2 "" H 1200 1950 50  0001 C CNN
@@
 AR Path="/6161C99E" Ref="C?"  Part="1"
 AR Path="/615A5F2C/6161C99E" Ref="C4"  Part="1"
-F 0 "C?" H 1315 1746 50  0000 L CNN
+F 0 "C4" H 1315 1746 50  0000 L CNN
 F 1 "1uF" H 1315 1655 50  0000 L CNN
 F 2 "Capacitor_SMD:C_0603_1608Metric" H 1238 1550 50  0001 C CNN
@@
 AR Path="/6161C9A4" Ref="#PWR?"  Part="1"
 AR Path="/615A5F2C/6161C9A4" Ref="#PWR016"  Part="1"
-F 0 "#PWR?" H 1200 1300 50  0001 C CNN
+F 0 "#PWR016" H 1200 1300 50  0001 C CNN
 F 1 "+3.3V" H 1215 1623 50  0000 C CNN
 F 2 "" H 1200 1450 50  0001 C CNN
@@
 AR Path="/6161C9AC" Ref="C?"  Part="1"
 AR Path="/615A5F2C/6161C9AC" Ref="C5"  Part="1"
-F 0 "C?" H 1715 1746 50  0000 L CNN
+F 0 "C5" H 1715 1746 50  0000 L CNN
 F 1 "100nF" H 1715 1655 50  0000 L CNN
 F 2 "Capacitor_SMD:C_0603_1608Metric" H 1638 1550 50  0001 C CNN
@@
 AR Path="/6161C9B2" Ref="C?"  Part="1"
 AR Path="/615A5F2C/6161C9B2" Ref="C6"  Part="1"
-F 0 "C?" H 2165 1746 50  0000 L CNN
+F 0 "C6" H 2165 1746 50  0000 L CNN
 F 1 "100nF" H 2165 1655 50  0000 L CNN
 F 2 "Capacitor_SMD:C_0603_1608Metric" H 2088 1550 50  0001 C CNN
@@
 AR Path="/6161C9B8" Ref="C?"  Part="1"
 AR Path="/615A5F2C/6161C9B8" Ref="C7"  Part="1"
-F 0 "C?" H 2615 1746 50  0000 L CNN
+F 0 "C7" H 2615 1746 50  0000 L CNN
 F 1 "100nF" H 2615 1655 50  0000 L CNN
 F 2 "Capacitor_SMD:C_0603_1608Metric" H 2538 1550 50  0001 C CNN
@@
 AR Path="/6161C9D2" Ref="C?"  Part="1"
 AR Path="/615A5F2C/6161C9D2" Ref="C8"  Part="1"
-F 0 "C?" H 3065 1746 50  0000 L CNN
+F 0 "C8" H 3065 1746 50  0000 L CNN
 F 1 "100nF" H 3065 1655 50  0000 L CNN
 F 2 "Capacitor_SMD:C_0603_1608Metric" H 2988 1550 50  0001 C CNN
@@
 AR Path="/61679BC7" Ref="#PWR?"  Part="1"
 AR Path="/615A5F2C/61679BC7" Ref="#PWR023"  Part="1"
-F 0 "#PWR?" H 9400 3150 50  0001 C CNN
+F 0 "#PWR023" H 9400 3150 50  0001 C CNN
 F 1 "GND" H 9405 3227 50  0000 C CNN
 F 2 "" H 9400 3400 50  0001 C CNN
@@
 AR Path="/6167BBB2" Ref="#PWR?"  Part="1"
 AR Path="/615A5F2C/6167BBB2" Ref="#PWR020"  Part="1"
-F 0 "#PWR?" H 6550 3450 50  0001 C CNN
+F 0 "#PWR020" H 6550 3450 50  0001 C CNN
 F 1 "GND" H 6555 3527 50  0000 C CNN
 F 2 "" H 6550 3700 50  0001 C CNN
@@
 AR Path="/6161C986" Ref="U?"  Part="1"
 AR Path="/615A5F2C/6161C986" Ref="U4"  Part="1"
-F 0 "U?" H 7700 4300 50  0000 C CNN
+F 0 "U4" H 7700 4300 50  0000 C CNN
 F 1 "MAX-8Q" H 7700 4200 50  0000 C CNN
 F 2 "RF_GPS:ublox_MAX" H 8100 2550 50  0001 C CNN
@@
 AR Path="/616192D0" Ref="L?"  Part="1"
 AR Path="/615A5F2C/616192D0" Ref="L1"  Part="1"
-F 0 "L?" H 3703 5996 50  0000 L CNN
+AR Path="/61E8EFE4/616192D0" Ref="L1"  Part="1"
+F 0 "L1" H 3703 5996 50  0000 L CNN
 F 1 "27nH" H 3703 5905 50  0000 L CNN
-F 2 "Inductor_THT:L_Radial_D10.5mm_P5.00mm_Abacron_AISR-01" H 3650 5950 50  0001 C CNN
+F 2 "Inductor_SMD:L_0603_1608Metric" H 3650 5950 50  0001 C CNN
 F 3 "~" H 3650 5950 50  0001 C CNN
-F 4 "https://www.digikey.com/en/products/detail/abracon-llc/AIUR-04-273J/2343571" H 3650 5950 50  0001 C CNN "Digikey"
+F 4 "https://www.digikey.com/en/products/detail/murata-electronics/LQG15HS27NJ02D/662877" H 3650 5950 50  0001 C CNN "Digikey"
+F 5 "LQG15HS27NJ02" H 3650 5950 50  0001 C CNN "Field5"
 	1    3650 5950
 	-1   0    0    -1
@@
 AR Path="/61619311" Ref="R?"  Part="1"
 AR Path="/615A5F2C/61619311" Ref="R3"  Part="1"
-F 0 "R?" H 3720 5596 50  0000 L CNN
+F 0 "R3" H 3720 5596 50  0000 L CNN
 F 1 "10k" H 3720 5505 50  0000 L CNN
 F 2 "Resistor_SMD:R_0603_1608Metric" V 3580 5550 50  0001 C CNN
@@
 AR Path="/616192EF" Ref="Q?"  Part="1"
 AR Path="/615A5F2C/616192EF" Ref="Q1"  Part="1"
-F 0 "Q?" H 4000 6192 50  0000 C CNN
+F 0 "Q1" H 4000 6192 50  0000 C CNN
 F 1 "SI1040X-T1-GE3" H 4000 6101 50  0000 C CNN
 F 2 "SC-89:SC-89" H 3950 5075 50  0001 C CNN

Commit message: Schematic Tweaks and Board Dimensioned
Parts:
- C4, C5, C6, C7, C8, C9: footprint Capacitor_SMD:C_0603_1608Metric -> Capacitor_SMD:C_0603_1608Metric_Pad1.08x0.95mm_HandSolder
- L1: footprint Inductor_SMD:L_0603_1608Metric -> Capacitor_SMD:C_0603_1608Metric_Pad1.08x0.95mm_HandSolder
- R3, R4, R5: footprint Resistor_SMD:R_0603_1608Metric -> Resistor_SMD:R_0603_1608Metric_Pad0.98x0.95mm_HandSolder
Changed lines of the file:
@@
 F 0 "C9" H 5015 5596 50  0000 L CNN
 F 1 "1nF" H 5015 5505 50  0000 L CNN
-F 2 "Capacitor_SMD:C_0603_1608Metric" H 4938 5400 50  0001 C CNN
+F 2 "Capacitor_SMD:C_0603_1608Metric_Pad1.08x0.95mm_HandSolder" H 4938 5400 50  0001 C CNN
 F 3 "~" H 4900 5550 50  0001 C CNN
 	1    4900 5550
@@
 F 0 "R5" H 4770 5596 50  0000 L CNN
 F 1 "100k" H 4770 5505 50  0000 L CNN
-F 2 "Resistor_SMD:R_0603_1608Metric" V 4630 5550 50  0001 C CNN
+F 2 "Resistor_SMD:R_0603_1608Metric_Pad0.98x0.95mm_HandSolder" V 4630 5550 50  0001 C CNN
 F 3 "~" H 4700 5550 50  0001 C CNN
 	1    4700 5550
@@
 F 0 "R4" H 4420 6296 50  0000 L CNN
 F 1 "10k" H 4420 6205 50  0000 L CNN
-F 2 "Resistor_SMD:R_0603_1608Metric" V 4280 6250 50  0001 C CNN
+F 2 "Resistor_SMD:R_0603_1608Metric_Pad0.98x0.95mm_HandSolder" V 4280 6250 50  0001 C CNN
 F 3 "~" H 4350 6250 50  0001 C CNN
 	1    4350 6250
@@
 F 0 "C4" H 1315 1746 50  0000 L CNN
 F 1 "1uF" H 1315 1655 50  0000 L CNN
-F 2 "Capacitor_SMD:C_0603_1608Metric" H 1238 1550 50  0001 C CNN
+F 2 "Capacitor_SMD:C_0603_1608Metric_Pad1.08x0.95mm_HandSolder" H 1238 1550 50  0001 C CNN
 F 3 "~" H 1200 1700 50  0001 C CNN
 	1    1200 1700
@@
 F 0 "C5" H 1715 1746 50  0000 L CNN
 F 1 "100nF" H 1715 1655 50  0000 L CNN
-F 2 "Capacitor_SMD:C_0603_1608Metric" H 1638 1550 50  0001 C CNN
+F 2 "Capacitor_SMD:C_0603_1608Metric_Pad1.08x0.95mm_HandSolder" H 1638 1550 50  0001 C CNN
 F 3 "~" H 1600 1700 50  0001 C CNN
 	1    1600 1700
@@
 F 0 "C6" H 2165 1746 50  0000 L CNN
 F 1 "100nF" H 2165 1655 50  0000 L CNN
-F 2 "Capacitor_SMD:C_0603_1608Metric" H 2088 1550 50  0001 C CNN
+F 2 "Capacitor_SMD:C_0603_1608Metric_Pad1.08x0.95mm_HandSolder" H 2088 1550 50  0001 C CNN
 F 3 "~" H 2050 1700 50  0001 C CNN
 	1    2050 1700
@@
 F 0 "C7" H 2615 1746 50  0000 L CNN
 F 1 "100nF" H 2615 1655 50  0000 L CNN
-F 2 "Capacitor_SMD:C_0603_1608Metric" H 2538 1550 50  0001 C CNN
+F 2 "Capacitor_SMD:C_0603_1608Metric_Pad1.08x0.95mm_HandSolder" H 2538 1550 50  0001 C CNN
 F 3 "~" H 2500 1700 50  0001 C CNN
 	1    2500 1700
@@
 F 0 "C8" H 3065 1746 50  0000 L CNN
 F 1 "100nF" H 3065 1655 50  0000 L CNN
-F 2 "Capacitor_SMD:C_0603_1608Metric" H 2988 1550 50  0001 C CNN
+F 2 "Capacitor_SMD:C_0603_1608Metric_Pad1.08x0.95mm_HandSolder" H 2988 1550 50  0001 C CNN
 F 3 "~" H 2950 1700 50  0001 C CNN
 	1    2950 1700
@@
 F 0 "L1" H 3703 5996 50  0000 L CNN
 F 1 "27nH" H 3703 5905 50  0000 L CNN
-F 2 "Inductor_SMD:L_0603_1608Metric" H 3650 5950 50  0001 C CNN
+F 2 "Capacitor_SMD:C_0603_1608Metric_Pad1.08x0.95mm_HandSolder" H 3650 5950 50  0001 C CNN
 F 3 "~" H 3650 5950 50  0001 C CNN
 F 4 "https://www.digikey.com/en/products/detail/murata-electronics/LQG15HS27NJ02D/662877" H 3650 5950 50  0001 C CNN "Digikey"
@@
 F 0 "R3" H 3720 5596 50  0000 L CNN
 F 1 "10k" H 3720 5505 50  0000 L CNN
-F 2 "Resistor_SMD:R_0603_1608Metric" V 3580 5550 50  0001 C CNN
+F 2 "Resistor_SMD:R_0603_1608Metric_Pad0.98x0.95mm_HandSolder" V 3580 5550 50  0001 C CNN
 F 3 "~" H 3650 5550 50  0001 C CNN
 	1    3650 5550

Commit message: finished routing
Parts:
- removed C6: 100nF, Capacitor_SMD:C_0603_1608Metric_Pad1.08x0.95mm_HandSolder, symbol Data_Collection_KiCAD_Project-rescue:C-Device-Data_Collection_KiCAD_Project-res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
Connections:
- wire segments 62 -> 58
Changed lines of the file:
@@
-$Comp
-L Data_Collection_KiCAD_Project-rescue:C-Device-Data_Collection_KiCAD_Project-rescue C?
-U 1 1 6161C9B2
-P 2050 1700
-AR Path="/6161C9B2" Ref="C?"  Part="1"
-AR Path="/615A5F2C/6161C9B2" Ref="C6"  Part="1"
-F 0 "C6" H 2165 1746 50  0000 L CNN
-F 1 "100nF" H 2165 1655 50  0000 L CNN
-F 2 "Capacitor_SMD:C_0603_1608Metric_Pad1.08x0.95mm_HandSolder" H 2088 1550 50  0001 C CNN
-F 3 "~" H 2050 1700 50  0001 C CNN
-	1    2050 1700
-	1    0    0    -1
-$EndComp
 $Comp
 L Data_Collection_KiCAD_Project-rescue:C-Device-Data_Collection_KiCAD_Project-rescue C?
@@
 Wire Wire Line
 	2500 1550 2500 1500
-Wire Wire Line
-	2500 1500 2050 1500
 Connection ~ 1200 1500
 Wire Wire Line
@@
 	1600 1500 1200 1500
 Wire Wire Line
-	2050 1550 2050 1500
-Connection ~ 2050 1500
-Wire Wire Line
-	2050 1500 1600 1500
-Wire Wire Line
-	2050 1850 2050 1900
-Connection ~ 2050 1900
-Wire Wire Line
-	2050 1900 2500 1900
-Wire Wire Line
 	1600 1850 1600 1900
 Connection ~ 1600 1900
-Wire Wire Line
-	1600 1900 2050 1900
 $Comp
 L Data_Collection_KiCAD_Project-rescue:C-Device-Data_Collection_KiCAD_Project-rescue C?
@@
 	-1   0    0    -1
 $EndComp
+Wire Wire Line
+	1600 1500 2500 1500
+Wire Wire Line
+	1600 1900 2500 1900
 $EndSCHEMATC
