File: Hardware/COMPONENT_SHEETS/MCU_STM32L562VET6Q.sch (KiCad schematic (older format))
At the start: 34 parts, among them Y1 32MHz

Commit message: GPS layout change and test point tweaks
Parts:
- removed JP?: VDDA Bridge, Jumper:SolderJumper-2_P1.3mm_Open_Pad1.0x1.5mm, symbol Jumper:SolderJumper_2_Open
- removed JP?: VDD_SMPS, Jumper:SolderJumper-2_P1.3mm_Open_Pad1.0x1.5mm, symbol Jumper:SolderJumper_2_Open
- IC1: renamed from IC?; symbol Charges_KiCAD_Project-rescue:STM32L562VET6Q-SamacSys_Parts -> Data_Collection_KiCAD_Project-rescue:STM32L562VET6Q-SamacSys_Parts-Charges_KiCAD_Project-rescue
- TP10, TP11, TP12, TP13, TP14, TP15, TP16, TP17, TP18, TP19, TP5, TP6, TP7, TP8, TP9: footprint Connector_PinHeader_1.00mm:PinHeader_1x01_P1.00mm_Vertical -> TestPoint:TestPoint_Loop_D1.80mm_Drill1.0mm_Beaded
- gave numbers to parts that had none: 6
Connections:
- wire segments 78 -> 76

Commit message: Schematic Tweaks and Board Dimensioned
Parts:
- removed TP10, TP11, TP12, TP13, TP17, TP18, TP19, TP5, TP6, TP7, TP8, TP9: Debug Pad, TestPoint:TestPoint_Loop_D1.80mm_Drill1.0mm_Beaded, symbol dk_Test-Points:RCT-0C
- added J4: I2C1 Debug, Connector_PinHeader_2.54mm:PinHeader_1x02_P2.54mm_Vertical, symbol Connector_Generic:Conn_01x02
- added J5: EXT I2c Debug, Connector_PinHeader_2.54mm:PinHeader_1x02_P2.54mm_Vertical, symbol Connector_Generic:Conn_01x02
- added J6: UART Debug, Connector_PinHeader_2.54mm:PinHeader_1x02_P2.54mm_Vertical, symbol Connector_Generic:Conn_01x02
- added J7: SPI 1 Debug, Connector_PinHeader_2.54mm:PinHeader_1x03_P2.54mm_Vertical, symbol Connector_Generic:Conn_01x03
- added J8: Ext SPI Debug, Connector_PinHeader_2.54mm:PinHeader_1x03_P2.54mm_Vertical, symbol Connector_Generic:Conn_01x03
- C10, C11, C12, C13, C14, C15, C16: footprint Capacitor_SMD:C_0603_1608Metric -> Capacitor_SMD:C_0603_1608Metric_Pad1.08x0.95mm_HandSolder
- D2, D3: footprint Diode_SMD:D_0603_1608Metric_Castellated -> Diode_SMD:D_0603_1608Metric_Pad1.05x0.95mm_HandSolder
- R10, R11, R6, R7, R8, R9: footprint Resistor_SMD:R_0603_1608Metric -> Resistor_SMD:R_0603_1608Metric_Pad0.98x0.95mm_HandSolder

Commit message: routing progress and pin reassignment
Parts:
- TP14, TP15, TP16: footprint TestPoint:TestPoint_Loop_D1.80mm_Drill1.0mm_Beaded -> TestPoint:TestPoint_Pad_D1.0mm
Changed lines of the file:
@@
 Text Notes 750  2400 0    50   ~ 0
 PVD_IN is the Power Voltage Dropout pin,\nused to detect and respond to brownout conditions.
-Text HLabel 6800 1500 1    50   Input ~ 0
+Text HLabel 9000 4000 2    50   Input ~ 0
 I2C1_SCL
-Text HLabel 6700 1500 1    50   Input ~ 0
+Text HLabel 9000 3900 2    50   Input ~ 0
 I2C1_SDA
-Text HLabel 9000 4700 2    50   Input ~ 0
+Text HLabel 6600 5700 3    50   Input ~ 0
 SPI2_SCK
 Text HLabel 8200 5700 3    50   Input ~ 0
@@
 Text HLabel 8100 5700 3    50   Input ~ 0
 EXT_SCL
-Text HLabel 9000 4600 2    50   Input ~ 0
+Text HLabel 6700 5700 3    50   Input ~ 0
 SPI2_MISO
-Text HLabel 9000 4500 2    50   Input ~ 0
+Text HLabel 6800 5700 3    50   Input ~ 0
 SPI2_MOSI
-Text HLabel 6600 5700 3    50   Input ~ 0
+Text HLabel 8500 1500 1    50   Input ~ 0
 SPI1_SCK
 Text HLabel 9000 3100 2    50   Input ~ 0
@@
 Text HLabel 9000 3000 2    50   Input ~ 0
 USART2_RX
-Text HLabel 6700 5700 3    50   Input ~ 0
+Text HLabel 8400 1500 1    50   Input ~ 0
 SPI1_MISO
-Text HLabel 6800 5700 3    50   Input ~ 0
+Text HLabel 8300 1500 1    50   Input ~ 0
 SPI1_MOSI
 Text HLabel 9000 2900 2    50   Input ~ 0
@@
 F 0 "TP15" V 9100 3500 50  0000 C CNN
 F 1 "Debug Pad" V 8966 3647 50  0001 C CNN
-F 2 "TestPoint:TestPoint_Loop_D1.80mm_Drill1.0mm_Beaded" H 9300 3800 60  0001 L CNN
+F 2 "TestPoint:TestPoint_Pad_D1.0mm" H 9300 3800 60  0001 L CNN
 F 3 "https://www.te.com/commerce/DocumentDelivery/DDEController?Action=srchrtrv&DocNm=1773266&DocType=DS&DocLang=English" H 9300 3900 60  0001 L CNN
 F 4 "A106144CT-ND" H 9300 4000 60  0001 L CNN "Digi-Key_PN"
@@
 F 0 "TP16" V 9100 3600 50  0000 C CNN
 F 1 "Debug Pad" V 8966 3747 50  0001 C CNN
-F 2 "TestPoint:TestPoint_Loop_D1.80mm_Drill1.0mm_Beaded" H 9300 3900 60  0001 L CNN
+F 2 "TestPoint:TestPoint_Pad_D1.0mm" H 9300 3900 60  0001 L CNN
 F 3 "https://www.te.com/commerce/DocumentDelivery/DDEController?Action=srchrtrv&DocNm=1773266&DocType=DS&DocLang=English" H 9300 4000 60  0001 L CNN
 F 4 "A106144CT-ND" H 9300 4100 60  0001 L CNN "Digi-Key_PN"
@@
 F 0 "TP14" V 9100 3400 50  0000 C CNN
 F 1 "Debug Pad" V 8966 3547 50  0001 C CNN
-F 2 "TestPoint:TestPoint_Loop_D1.80mm_Drill1.0mm_Beaded" H 9300 3700 60  0001 L CNN
+F 2 "TestPoint:TestPoint_Pad_D1.0mm" H 9300 3700 60  0001 L CNN
 F 3 "https://www.te.com/commerce/DocumentDelivery/DDEController?Action=srchrtrv&DocNm=1773266&DocType=DS&DocLang=English" H 9300 3800 60  0001 L CNN
 F 4 "A106144CT-ND" H 9300 3900 60  0001 L CNN "Digi-Key_PN"

Commit message: finished routing
Parts:
- removed J5: EXT I2c Debug, Connector_PinHeader_2.54mm:PinHeader_1x02_P2.54mm_Vertical, symbol Connector_Generic:Conn_01x02
- removed J8: Ext SPI Debug, Connector_PinHeader_2.54mm:PinHeader_1x03_P2.54mm_Vertical, symbol Connector_Generic:Conn_01x03
- removed TP14, TP15, TP16: Debug Pad, TestPoint:TestPoint_Pad_D1.0mm, symbol dk_Test-Points:RCT-0C
Changed lines of the file:
@@
 L Data_Collection_KiCAD_Project-rescue:LED-Device-Data_Collection_KiCAD_Project-rescue D?
 U 1 1 61E9E710
-P 4900 2500
+P 7250 6300
 AR Path="/61E9E710" Ref="D?"  Part="1"
 AR Path="/61E8EFE4/61E9E710" Ref="D2"  Part="1"
-F 0 "D2" V 4939 2382 50  0000 R CNN
-F 1 "Green" V 4848 2382 50  0000 R CNN
-F 2 "Diode_SMD:D_0603_1608Metric_Pad1.05x0.95mm_HandSolder" H 4900 2500 50  0001 C CNN
-F 3 "https://fscdn.rohm.com/en/products/databook/datasheet/opto/led/chip_mono/sml-d12x8_d13x8-e.pdf" H 4900 2500 50  0001 C CNN
-F 4 "https://www.digikey.com/en/products/detail/rohm-semiconductor/SML-D12P8WT86/1641798" V 4900 2500 50  0001 C CNN "Digikey"
-	1    4900 2500
+F 0 "D2" V 7289 6182 50  0000 R CNN
+F 1 "Green" V 7198 6182 50  0000 R CNN
+F 2 "Diode_SMD:D_0603_1608Metric_Pad1.05x0.95mm_HandSolder" H 7250 6300 50  0001 C CNN
+F 3 "https://fscdn.rohm.com/en/products/databook/datasheet/opto/led/chip_mono/sml-d12x8_d13x8-e.pdf" H 7250 6300 50  0001 C CNN
+F 4 "https://www.digikey.com/en/products/detail/rohm-semiconductor/SML-D12P8WT86/1641798" V 7250 6300 50  0001 C CNN "Digikey"
+	1    7250 6300
 	1    0    0    -1
 $EndComp
@@
 L Device:R_US R10
 U 1 1 619EFD59
-P 5200 2500
-F 0 "R10" H 5268 2546 50  0000 L CNN
-F 1 "80" H 5268 2455 50  0000 L CNN
-F 2 "Resistor_SMD:R_0603_1608Metric_Pad0.98x0.95mm_HandSolder" V 5240 2490 50  0001 C CNN
-F 3 "~" H 5200 2500 50  0001 C CNN
-	1    5200 2500
-	0    1    1    0
-$EndComp
-$Comp
-L Device:R_US R11
-U 1 1 619F2A76
 P 7400 6000
-F 0 "R11" H 7468 6046 50  0000 L CNN
+F 0 "R10" H 7468 6046 50  0000 L CNN
 F 1 "80" H 7468 5955 50  0000 L CNN
 F 2 "Resistor_SMD:R_0603_1608Metric_Pad0.98x0.95mm_HandSolder" V 7440 5990 50  0001 C CNN
@@
 $EndComp
 $Comp
+L Device:R_US R11
+U 1 1 619F2A76
+P 5100 2500
+F 0 "R11" H 5168 2546 50  0000 L CNN
+F 1 "80" H 5168 2455 50  0000 L CNN
+F 2 "Resistor_SMD:R_0603_1608Metric_Pad0.98x0.95mm_HandSolder" V 5140 2490 50  0001 C CNN
+F 3 "~" H 5100 2500 50  0001 C CNN
+	1    5100 2500
+	0    1    1    0
+$EndComp
+$Comp
 L Data_Collection_KiCAD_Project-rescue:LED-Device-Data_Collection_KiCAD_Project-rescue D?
 U 1 1 619F2F50
-P 7250 6300
+P 4800 2500
 AR Path="/619F2F50" Ref="D?"  Part="1"
 AR Path="/61E8EFE4/619F2F50" Ref="D3"  Part="1"
-F 0 "D3" H 7300 6150 50  0000 R CNN
-F 1 "Red" H 7200 6400 50  0000 R CNN
-F 2 "Diode_SMD:D_0603_1608Metric_Pad1.05x0.95mm_HandSolder" H 7250 6300 50  0001 C CNN
-F 3 "https://fscdn.rohm.com/en/products/databook/datasheet/opto/led/chip_mono/sml-d12x8_d13x8-e.pdf" H 7250 6300 50  0001 C CNN
-F 4 "https://www.digikey.com/en/products/detail/rohm-semiconductor/SML-D12U8WT86/1641799" V 7250 6300 50  0001 C CNN "Digikey"
-	1    7250 6300
+F 0 "D3" H 4850 2350 50  0000 R CNN
+F 1 "Red" H 4850 2250 50  0000 R CNN
+F 2 "Diode_SMD:D_0603_1608Metric_Pad1.05x0.95mm_HandSolder" H 4800 2500 50  0001 C CNN
+F 3 "https://fscdn.rohm.com/en/products/databook/datasheet/opto/led/chip_mono/sml-d12x8_d13x8-e.pdf" H 4800 2500 50  0001 C CNN
+F 4 "https://www.digikey.com/en/products/detail/rohm-semiconductor/SML-D12U8WT86/1641799" V 4800 2500 50  0001 C CNN "Digikey"
+	1    4800 2500
 	1    0    0    -1
 $EndComp
@@
 Text HLabel 1150 7000 2    50   Input ~ 0
 I2C1_SDA
-Text HLabel 1150 7350 2    50   Input ~ 0
-EXT_SCL
-Text HLabel 1150 7450 2    50   Input ~ 0
-EXT_SDA
 Wire Notes Line
 	1650 7550 650  7550
@@
 	9000 4800 10500 4800
 Wire Wire Line
-	6000 2500 5350 2500
-Wire Wire Line
-	4750 2500 4500 2500
-Wire Wire Line
 	4500 2500 4500 2650
 Wire Wire Line
@@
 Wire Wire Line
 	7400 5850 7400 5700
-$Comp
-L dk_Test-Points:RCT-0C TP?
-U 1 1 61B55D71
-P 9100 3600
-AR Path="/61B55D71" Ref="TP?"  Part="1"
-AR Path="/61E8EFE4/61B55D71" Ref="TP15"  Part="1"
-F 0 "TP15" V 9100 3500 50  0000 C CNN
-F 1 "Debug Pad" V 8966 3647 50  0001 C CNN
-F 2 "TestPoint:TestPoint_Pad_D1.0mm" H 9300 3800 60  0001 L CNN
-F 3 "https://www.te.com/commerce/DocumentDelivery/DDEController?Action=srchrtrv&DocNm=1773266&DocType=DS&DocLang=English" H 9300 3900 60  0001 L CNN
-F 4 "A106144CT-ND" H 9300 4000 60  0001 L CNN "Digi-Key_PN"
-F 5 "RCT-0C" H 9300 4100 60  0001 L CNN "MPN"
-F 6 "Test and Measurement" H 9300 4200 60  0001 L CNN "Category"
-F 7 "Test Points" H 9300 4300 60  0001 L CNN "Family"
-F 8 "https://www.te.com/commerce/DocumentDelivery/DDEController?Action=srchrtrv&DocNm=1773266&DocType=DS&DocLang=English" H 9300 4400 60  0001 L CNN "DK_Datasheet_Link"
-F 9 "/product-detail/en/te-connectivity-amp-connectors/RCT-0C/A106144CT-ND/3477801" H 9300 4500 60  0001 L CNN "DK_Detail_Page"
-F 10 "PC TEST POINT NATURAL" H 9300 4600 60  0001 L CNN "Description"
-F 11 "TE Connectivity AMP Connectors" H 9300 4700 60  0001 L CNN "Manufacturer"
-F 12 "Active" H 9300 4800 60  0001 L CNN "Status"
-	1    9100 3600
-	0    -1   -1   0
-$EndComp
-$Comp
-L dk_Test-Points:RCT-0C TP?
-U 1 1 61B5C473
-P 9100 3700
-AR Path="/61B5C473" Ref="TP?"  Part="1"
-AR Path="/61E8EFE4/61B5C473" Ref="TP16"  Part="1"
-F 0 "TP16" V 9100 3600 50  0000 C CNN
-F 1 "Debug Pad" V 8966 3747 50  0001 C CNN
-F 2 "TestPoint:TestPoint_Pad_D1.0mm" H 9300 3900 60  0001 L CNN
-F 3 "https://www.te.com/commerce/DocumentDelivery/DDEController?Action=srchrtrv&DocNm=1773266&DocType=DS&DocLang=English" H 9300 4000 60  0001 L CNN
-F 4 "A106144CT-ND" H 9300 4100 60  0001 L CNN "Digi-Key_PN"
-F 5 "RCT-0C" H 9300 4200 60  0001 L CNN "MPN"
-F 6 "Test and Measurement" H 9300 4300 60  0001 L CNN "Category"
-F 7 "Test Points" H 9300 4400 60  0001 L CNN "Family"
-F 8 "https://www.te.com/commerce/DocumentDelivery/DDEController?Action=srchrtrv&DocNm=1773266&DocType=DS&DocLang=English" H 9300 4500 60  0001 L CNN "DK_Datasheet_Link"
-F 9 "/product-detail/en/te-connectivity-amp-connectors/RCT-0C/A106144CT-ND/3477801" H 9300 4600 60  0001 L CNN "DK_Detail_Page"
-F 10 "PC TEST POINT NATURAL" H 9300 4700 60  0001 L CNN "Description"
-F 11 "TE Connectivity AMP Connectors" H 9300 4800 60  0001 L CNN "Manufacturer"
-F 12 "Active" H 9300 4900 60  0001 L CNN "Status"
-	1    9100 3700
-	0    -1   -1   0
-$EndComp
-$Comp
-L dk_Test-Points:RCT-0C TP?
-U 1 1 61B5C94C
-P 9100 3500
-AR Path="/61B5C94C" Ref="TP?"  Part="1"
-AR Path="/61E8EFE4/61B5C94C" Ref="TP14"  Part="1"
-F 0 "TP14" V 9100 3400 50  0000 C CNN
-F 1 "Debug Pad" V 8966 3547 50  0001 C CNN
-F 2 "TestPoint:TestPoint_Pad_D1.0mm" H 9300 3700 60  0001 L CNN
-F 3 "https://www.te.com/commerce/DocumentDelivery/DDEController?Action=srchrtrv&DocNm=1773266&DocType=DS&DocLang=English" H 9300 3800 60  0001 L CNN
-F 4 "A106144CT-ND" H 9300 3900 60  0001 L CNN "Digi-Key_PN"
-F 5 "RCT-0C" H 9300 4000 60  0001 L CNN "MPN"
-F 6 "Test and Measurement" H 9300 4100 60  0001 L CNN "Category"
-F 7 "Test Points" H 9300 4200 60  0001 L CNN "Family"
-F 8 "https://www.te.com/commerce/DocumentDelivery/DDEController?Action=srchrtrv&DocNm=1773266&DocType=DS&DocLang=English" H 9300 4300 60  0001 L CNN "DK_Datasheet_Link"
-F 9 "/product-detail/en/te-connectivity-amp-connectors/RCT-0C/A106144CT-ND/3477801" H 9300 4400 60  0001 L CNN "DK_Detail_Page"
-F 10 "PC TEST POINT NATURAL" H 9300 4500 60  0001 L CNN "Description"
-F 11 "TE Connectivity AMP Connectors" H 9300 4600 60  0001 L CNN "Manufacturer"
-F 12 "Active" H 9300 4700 60  0001 L CNN "Status"
-	1    9100 3500
-	0    -1   -1   0
-$EndComp
 Wire Notes Line
 	3650 6750 4550 6750
@@
 Text Notes 3650 6700 0    50   ~ 0
 SPI 2  Debug
-Text HLabel 4050 7100 2    50   Input ~ 0
-SPI2_SCK
-Text HLabel 4050 7300 2    50   Input ~ 0
-SPI2_MOSI
-Text HLabel 4050 7200 2    50   Input ~ 0
-SPI2_MISO
 $Comp
 L Data_Collection_KiCAD_Project-rescue:STM32L562VET6Q-SamacSys_Parts-Charges_KiCAD_Project-rescue IC1
@@
 	7650 6450 8300 6450
 $Comp
-L Connector_Generic:Conn_01x03 J8
-U 1 1 61C1F908
-P 3850 7200
-F 0 "J8" H 3768 6875 50  0000 C CNN
-F 1 "Ext SPI Debug" H 3768 6966 50  0000 C CNN
-F 2 "Connector_PinHeader_2.54mm:PinHeader_1x03_P2.54mm_Vertical" H 3850 7200 50  0001 C CNN
-F 3 "~" H 3850 7200 50  0001 C CNN
-	1    3850 7200
-	-1   0    0    1
-$EndComp
-$Comp
 L Connector_Generic:Conn_01x03 J7
 U 1 1 61C20D7F
@@
 Text Notes 650  6500 0    50   ~ 0
 I2C Debug Pts
-$Comp
-L Connector_Generic:Conn_01x02 J5
-U 1 1 61C2C82E
-P 950 7450
-F 0 "J5" H 868 7125 50  0000 C CNN
-F 1 "EXT I2c Debug" H 868 7216 50  0000 C CNN
-F 2 "Connector_PinHeader_2.54mm:PinHeader_1x02_P2.54mm_Vertical" H 950 7450 50  0001 C CNN
-F 3 "~" H 950 7450 50  0001 C CNN
-	1    950  7450
-	-1   0    0    1
-$EndComp
 Wire Notes Line
 	650  6550 650  7550
@@
 Wire Notes Line
 	650  5300 650  6150
+Wire Wire Line
+	5250 2500 6000 2500
+Wire Wire Line
+	4650 2500 4500 2500
 $EndSCHEMATC
