File: Hardware/COMPONENT_SHEETS/MCU_L562VE.kicad_sch (KiCad schematic)
At the start: 29 parts

Commit message: Corrected PCB edge cuts, removed components
Will be mimicking layout done by Seth Sievers
Parts:
- gave numbers to parts that had none: 29
Connections:
- net ~{USART2_RST}: now reaches U9.67 (PA8)
- no-connect marks 47 -> 46
