File: Hardware/COMPONENT_SHEETS/BAROMETER_MS5607-02.kicad_sch (KiCad schematic)
At the start: 2 parts, among them U7 MS5607-02BA

Commit message: Corrected PCB edge cuts, removed components
Will be mimicking layout done by Seth Sievers
Parts:
- renumbered C18 to C12
Changed lines of the file:
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@@
   (symbol (lib_id "Data_Collection_KiCAD_Project-rescue:+3.3V-power-Data_Collection_KiCAD_Project-rescue") (at 161.29 80.01 0)
     (in_bom yes) (on_board yes)
-    (property "Reference" "#PWR040" (id 0) (at 161.29 83.82 0)
+    (property "Reference" "#PWR041" (id 0) (at 161.29 83.82 0)
       (effects (font (size 1.27 1.27)) hide)
     )
@@
   (symbol (lib_id "Data_Collection_KiCAD_Project-rescue:GND-power-Data_Collection_KiCAD_Project-rescue") (at 149.86 105.41 0)
     (in_bom yes) (on_board yes)
-    (property "Reference" "#PWR039" (id 0) (at 149.86 111.76 0)
+    (property "Reference" "#PWR040" (id 0) (at 149.86 111.76 0)
       (effects (font (size 1.27 1.27)) hide)
     )
@@
   (symbol (lib_id "Data_Collection_KiCAD_Project-rescue:C-Device-Data_Collection_KiCAD_Project-rescue") (at 161.29 92.71 0)
     (in_bom yes) (on_board yes)
-    (property "Reference" "C18" (id 0) (at 164.211 91.5416 0)
+    (property "Reference" "C12" (id 0) (at 164.211 91.5416 0)
       (effects (font (size 1.27 1.27)) (justify left))
     )
