File: Hardware/COMPONENT_SHEETS/FLASH_W25Q32JV.kicad_sch (KiCad schematic)
At the start: 1 part, among them U6 W25Q32JVSS

Commit message: Updated MCU Component Sheet
Used the file from the Telemetry board for compatibility and commonality.
Changed lines of the file:
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@@
     (comment 3 "Schematic depicting logical connections between components")
-  )
-  (junction (at 105.41 69.85) (diameter 0) (color 0 0 0 0)
   )
   (junction (at 139.7 86.36) (diameter 0) (color 0 0 0 0)
   )
   (wire (pts (xy 125.73 71.12) (xy 125.73 69.85))
-    (stroke (width 0) (type default) (color 0 0 0 0))
-  )
-  (wire (pts (xy 97.79 69.85) (xy 105.41 69.85))
     (stroke (width 0) (type default) (color 0 0 0 0))
   )
@@
     (stroke (width 0) (type default) (color 0 0 0 0))
   )
-  (wire (pts (xy 97.79 76.2) (xy 97.79 69.85))
-    (stroke (width 0) (type default) (color 0 0 0 0))
-  )

Commit message: Corrected PCB edge cuts, removed components
Will be mimicking layout done by Seth Sievers
Parts:
- renumbered U6 to U2
Changed lines of the file:
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@@
   (symbol (lib_id "Data_Collection_KiCAD_Project-rescue:W25Q32JVSS-Memory_Flash-Data_Collection_KiCAD_Project-rescue") (at 125.73 81.28 0)
     (in_bom yes) (on_board yes)
-    (property "Reference" "U6" (id 0) (at 125.73 60.96 0))
+    (property "Reference" "U2" (id 0) (at 125.73 60.96 0))
     (property "Value" "W25Q32JVSS" (id 1) (at 125.73 63.5 0))
     (property "Footprint" "Package_SO:SOIC-8_5.23x5.23mm_P1.27mm" (id 2) (at 125.73 81.28 0)
@@
   (symbol (lib_id "Data_Collection_KiCAD_Project-rescue:+3.3V-power-Data_Collection_KiCAD_Project-rescue") (at 105.41 68.58 0)
     (in_bom yes) (on_board yes)
-    (property "Reference" "#PWR036" (id 0) (at 105.41 72.39 0)
+    (property "Reference" "#PWR018" (id 0) (at 105.41 72.39 0)
       (effects (font (size 1.27 1.27)) hide)
     )
@@
   (symbol (lib_id "Data_Collection_KiCAD_Project-rescue:GND-power-Data_Collection_KiCAD_Project-rescue") (at 125.73 91.44 0)
     (in_bom yes) (on_board yes)
-    (property "Reference" "#PWR037" (id 0) (at 125.73 97.79 0)
+    (property "Reference" "#PWR019" (id 0) (at 125.73 97.79 0)
       (effects (font (size 1.27 1.27)) hide)
     )
@@
   (symbol (lib_id "Data_Collection_KiCAD_Project-rescue:GND-power-Data_Collection_KiCAD_Project-rescue") (at 139.7 87.63 0)
     (in_bom yes) (on_board yes)
-    (property "Reference" "#PWR038" (id 0) (at 139.7 93.98 0)
+    (property "Reference" "#PWR020" (id 0) (at 139.7 93.98 0)
       (effects (font (size 1.27 1.27)) hide)
     )

Commit message: Organized components, arranged filter caps
Parts:
- added C30: 0.1uF, Capacitor_SMD:C_0603_1608Metric_Pad1.08x0.95mm_HandSolder, symbol Data_Collection_KiCAD_Project-rescue:C_Small-Device-Data_Collection_KiCAD_Proje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
Connections:
- net +3V3: now also C30.1
- net GND: now also C30.2
Changed lines of the file:
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@@
     (comment 3 "Schematic depicting logical connections between components")
+  )
+  (junction (at 105.41 69.85) (diameter 0) (color 0 0 0 0)
   )
   (junction (at 139.7 86.36) (diameter 0) (color 0 0 0 0)
@@
     (effects (font (size 1.27 1.27)) (justify right))
   )
-  (symbol (lib_id "Data_Collection_KiCAD_Project-rescue:W25Q32JVSS-Memory_Flash-Data_Collection_KiCAD_Project-rescue") (at 125.73 81.28 0)
+  (symbol (lib_id "Data_Collection_KiCAD_Project-rescue:W25Q32JVSS-Memory_Flash-Data_Collection_KiCAD_Project-rescue") (at 125.73 81.28 0) (unit 1)
     (in_bom yes) (on_board yes)
     (property "Reference" "U2" (id 0) (at 125.73 60.96 0))
@@
     (pin "8")
   )
-  (symbol (lib_id "Data_Collection_KiCAD_Project-rescue:+3.3V-power-Data_Collection_KiCAD_Project-rescue") (at 105.41 68.58 0)
+  (symbol (lib_id "Data_Collection_KiCAD_Project-rescue:+3.3V-power-Data_Collection_KiCAD_Project-rescue") (at 105.41 68.58 0) (unit 1)
     (in_bom yes) (on_board yes)
     (property "Reference" "#PWR018" (id 0) (at 105.41 72.39 0)
@@
     (pin "1")
   )
-  (symbol (lib_id "Data_Collection_KiCAD_Project-rescue:GND-power-Data_Collection_KiCAD_Project-rescue") (at 125.73 91.44 0)
+  (symbol (lib_id "Data_Collection_KiCAD_Project-rescue:GND-power-Data_Collection_KiCAD_Project-rescue") (at 125.73 91.44 0) (unit 1)
     (in_bom yes) (on_board yes)
     (property "Reference" "#PWR019" (id 0) (at 125.73 97.79 0)
@@
     (pin "1")
   )
-  (symbol (lib_id "Data_Collection_KiCAD_Project-rescue:GND-power-Data_Collection_KiCAD_Project-rescue") (at 139.7 87.63 0)
+  (symbol (lib_id "Data_Collection_KiCAD_Project-rescue:GND-power-Data_Collection_KiCAD_Project-rescue") (at 139.7 87.63 0) (unit 1)
     (in_bom yes) (on_board yes)
     (property "Reference" "#PWR020" (id 0) (at 139.7 93.98 0)
@@
     (pin "1")
   )
+  (symbol (lib_id "Data_Collection_KiCAD_Project-rescue:GND-power-Data_Collection_KiCAD_Project-rescue") (at 105.41 74.93 0) (unit 1)
+    (in_bom yes) (on_board yes)
+    (property "Reference" "#PWR065" (id 0) (at 105.41 81.28 0)
+      (effects (font (size 1.27 1.27)) hide)
+    )
+    (property "Value" "GND" (id 1) (at 105.537 79.3242 0))
+    (property "Footprint" "" (id 2) (at 105.41 74.93 0)
+      (effects (font (size 1.27 1.27)) hide)
+    )
+    (property "Datasheet" "" (id 3) (at 105.41 74.93 0)
+      (effects (font (size 1.27 1.27)) hide)
+    )
+    (pin "1")
+  )
+  (symbol (lib_id "Data_Collection_KiCAD_Project-rescue:C_Small-Device-Data_Collection_KiCAD_Project-rescue") (at 105.41 72.39 0) (unit 1)
+    (in_bom yes) (on_board yes)
+    (property "Reference" "C30" (id 0) (at 99.5934 72.39 90))
+    (property "Value" "0.1uF" (id 1) (at 101.9048 72.39 90))
+    (property "Footprint" "Capacitor_SMD:C_0603_1608Metric_Pad1.08x0.95mm_HandSolder" (id 2) (at 105.41 72.39 0)
+      (effects (font (size 1.27 1.27)) hide)
+    )
+    (property "Datasheet" "~" (id 3) (at 105.41 72.39 0)
+      (effects (font (size 1.27 1.27)) hide)
+    )
+    (pin "1")
+    (pin "2")
+  )
 )
