File: Hardware/COMPONENT_SHEETS/TEMPSENSOR_MCP9808.kicad_sch (KiCad schematic)
At the start: 1 part, among them U3 MCP9808_MSOP

Commit message: Corrected PCB edge cuts, removed components
Will be mimicking layout done by Seth Sievers
Parts:
- renumbered U3 to U6
Changed lines of the file:
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@@
   (symbol (lib_id "Data_Collection_KiCAD_Project-rescue:MCP9808_MSOP-Sensor_Temperature-Data_Collection_KiCAD_Project-rescue") (at 139.7 90.17 0)
     (in_bom yes) (on_board yes)
-    (property "Reference" "U3" (id 0) (at 138.43 71.12 0)
+    (property "Reference" "U6" (id 0) (at 138.43 71.12 0)
       (effects (font (size 1.27 1.27)) (justify left))
     )
@@
   (symbol (lib_id "Data_Collection_KiCAD_Project-rescue:GND-power-Data_Collection_KiCAD_Project-rescue") (at 139.7 105.41 0)
     (in_bom yes) (on_board yes)
-    (property "Reference" "#PWR013" (id 0) (at 139.7 111.76 0)
+    (property "Reference" "#PWR038" (id 0) (at 139.7 111.76 0)
       (effects (font (size 1.27 1.27)) hide)
     )
@@
   (symbol (lib_id "Data_Collection_KiCAD_Project-rescue:+3.3V-power-Data_Collection_KiCAD_Project-rescue") (at 151.13 74.93 0)
     (in_bom yes) (on_board yes)
-    (property "Reference" "#PWR014" (id 0) (at 151.13 78.74 0)
+    (property "Reference" "#PWR039" (id 0) (at 151.13 78.74 0)
       (effects (font (size 1.27 1.27)) hide)
     )

Commit message: Organized components, arranged filter caps
Parts:
- added C29: 0.1uF, Capacitor_SMD:C_0603_1608Metric_Pad1.08x0.95mm_HandSolder, symbol Data_Collection_KiCAD_Project-rescue:C_Small-Device-Data_Collection_KiCAD_Proje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
Connections:
- net +3V3: now also C29.1
- net GND: now also C29.2
Changed lines of the file:
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@@
     (comment 3 "Schematic depicting logical connections between components")
+  )
+  (junction (at 151.13 76.2) (diameter 0) (color 0 0 0 0)
   )
   (polyline (pts (xy 118.11 68.58) (xy 118.11 111.76))
@@
     (effects (font (size 1.27 1.27)) (justify right))
   )
-  (symbol (lib_id "Data_Collection_KiCAD_Project-rescue:MCP9808_MSOP-Sensor_Temperature-Data_Collection_KiCAD_Project-rescue") (at 139.7 90.17 0)
+  (symbol (lib_id "Data_Collection_KiCAD_Project-rescue:MCP9808_MSOP-Sensor_Temperature-Data_Collection_KiCAD_Project-rescue") (at 139.7 90.17 0) (unit 1)
     (in_bom yes) (on_board yes)
     (property "Reference" "U6" (id 0) (at 138.43 71.12 0)
@@
     (pin "8")
   )
-  (symbol (lib_id "Data_Collection_KiCAD_Project-rescue:GND-power-Data_Collection_KiCAD_Project-rescue") (at 139.7 105.41 0)
+  (symbol (lib_id "Data_Collection_KiCAD_Project-rescue:GND-power-Data_Collection_KiCAD_Project-rescue") (at 139.7 105.41 0) (unit 1)
     (in_bom yes) (on_board yes)
     (property "Reference" "#PWR038" (id 0) (at 139.7 111.76 0)
@@
     (pin "1")
   )
-  (symbol (lib_id "Data_Collection_KiCAD_Project-rescue:+3.3V-power-Data_Collection_KiCAD_Project-rescue") (at 151.13 74.93 0)
+  (symbol (lib_id "Data_Collection_KiCAD_Project-rescue:+3.3V-power-Data_Collection_KiCAD_Project-rescue") (at 151.13 74.93 0) (unit 1)
     (in_bom yes) (on_board yes)
     (property "Reference" "#PWR039" (id 0) (at 151.13 78.74 0)
@@
       (effects (font (size 1.27 1.27)) hide)
     )
+    (pin "1")
+  )
+  (symbol (lib_id "Data_Collection_KiCAD_Project-rescue:C_Small-Device-Data_Collection_KiCAD_Project-rescue") (at 151.13 78.74 0) (unit 1)
+    (in_bom yes) (on_board yes)
+    (property "Reference" "C29" (id 0) (at 145.3134 78.74 90))
+    (property "Value" "0.1uF" (id 1) (at 147.6248 78.74 90))
+    (property "Footprint" "Capacitor_SMD:C_0603_1608Metric_Pad1.08x0.95mm_HandSolder" (id 2) (at 151.13 78.74 0)
+      (effects (font (size 1.27 1.27)) hide)
+    )
+    (property "Datasheet" "~" (id 3) (at 151.13 78.74 0)
+      (effects (font (size 1.27 1.27)) hide)
+    )
+    (pin "1")
+    (pin "2")
+  )
+  (symbol (lib_id "Data_Collection_KiCAD_Project-rescue:GND-power-Data_Collection_KiCAD_Project-rescue") (at 151.13 81.28 0) (unit 1)
+    (in_bom yes) (on_board yes)
+    (property "Reference" "#PWR064" (id 0) (at 151.13 87.63 0)
+      (effects (font (size 1.27 1.27)) hide)
+    )
+    (property "Value" "GND" (id 1) (at 151.257 85.6742 0))
+    (property "Footprint" "" (id 2) (at 151.13 81.28 0)
+      (effects (font (size 1.27 1.27)) hide)
+    )
+    (property "Datasheet" "" (id 3) (at 151.13 81.28 0)
+      (effects (font (size 1.27 1.27)) hide)
+    )
