File: Hardware/COMPONENT_SHEETS/USB_ESD.kicad_sch (KiCad schematic)
At the start: 9 parts, among them J1 10118192-0001LF, U5 USBLC6-2SC6

Commit message: Added 3D models to components
Parts:
- gave numbers to parts that had none: 6
Changed lines of the file:
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@@
   (symbol (lib_id "Device:R_Small") (at 138.43 97.79 270) (unit 1)
     (in_bom yes) (on_board yes)
-    (property "Reference" "R?" (id 0) (at 139.5984 99.2886 0)
+    (property "Reference" "R2" (id 0) (at 139.5984 99.2886 0)
       (effects (font (size 1.27 1.27)) (justify left))
     )
@@
   (symbol (lib_id "Device:D_Schottky_Small") (at 85.09 95.25 0) (mirror y) (unit 1)
     (in_bom yes) (on_board yes)
-    (property "Reference" "D?" (id 0) (at 85.09 90.043 0))
+    (property "Reference" "D1" (id 0) (at 85.09 90.043 0))
     (property "Value" "D_Schottky_Small" (id 1) (at 85.09 92.3544 0))
     (property "Footprint" "Diode_SMD:D_0603_1608Metric_Pad1.05x0.95mm_HandSolder" (id 2) (at 85.09 95.25 90)
@@
   (symbol (lib_id "Device:R_Small") (at 130.81 102.87 0) (unit 1)
     (in_bom yes) (on_board yes)
-    (property "Reference" "R?" (id 0) (at 132.3086 101.7016 0)
+    (property "Reference" "R1" (id 0) (at 132.3086 101.7016 0)
       (effects (font (size 1.27 1.27)) (justify left))
     )
@@
   (symbol (lib_id "power:GND") (at 97.79 102.87 0) (unit 1)
     (in_bom yes) (on_board yes)
-    (property "Reference" "#PWR?" (id 0) (at 97.79 109.22 0)
+    (property "Reference" "#PWR0129" (id 0) (at 97.79 109.22 0)
       (effects (font (size 1.27 1.27)) hide)
     )
@@
   (symbol (lib_id "power:+5V") (at 102.87 91.44 0) (unit 1)
     (in_bom yes) (on_board yes)
-    (property "Reference" "#PWR?" (id 0) (at 102.87 95.25 0)
+    (property "Reference" "#PWR0113" (id 0) (at 102.87 95.25 0)
       (effects (font (size 1.27 1.27)) hide)
     )
@@
   (symbol (lib_id "power:GND") (at 130.81 105.41 0) (unit 1)
     (in_bom yes) (on_board yes)
-    (property "Reference" "#PWR?" (id 0) (at 130.81 111.76 0)
+    (property "Reference" "#PWR0132" (id 0) (at 130.81 111.76 0)
       (effects (font (size 1.27 1.27)) hide)
     )
@@
   (symbol (lib_id "Device:C_Small") (at 144.78 102.87 0) (unit 1)
     (in_bom yes) (on_board yes)
-    (property "Reference" "C?" (id 0) (at 147.1168 101.7016 0)
+    (property "Reference" "C2" (id 0) (at 147.1168 101.7016 0)
       (effects (font (size 1.27 1.27)) (justify left))
     )
@@
   (symbol (lib_id "power:GND") (at 118.11 105.41 0) (unit 1)
     (in_bom yes) (on_board yes)
-    (property "Reference" "#PWR?" (id 0) (at 118.11 111.76 0)
+    (property "Reference" "#PWR0130" (id 0) (at 118.11 111.76 0)
       (effects (font (size 1.27 1.27)) hide)
     )
@@
   (symbol (lib_id "power:GND") (at 144.78 105.41 0) (unit 1)
     (in_bom yes) (on_board yes)
-    (property "Reference" "#PWR?" (id 0) (at 144.78 111.76 0)
+    (property "Reference" "#PWR0133" (id 0) (at 144.78 111.76 0)
       (effects (font (size 1.27 1.27)) hide)
     )
@@
   (symbol (lib_id "power:+3.3V") (at 133.35 91.44 0) (unit 1)
     (in_bom yes) (on_board yes)
-    (property "Reference" "#PWR?" (id 0) (at 133.35 95.25 0)
+    (property "Reference" "#PWR0131" (id 0) (at 133.35 95.25 0)
       (effects (font (size 1.27 1.27)) hide)
     )
@@
   (symbol (lib_id "Regulator_Linear:ADP7182AUJZ") (at 118.11 97.79 0) (mirror x) (unit 1)
     (in_bom yes) (on_board yes) (fields_autoplaced)
-    (property "Reference" "U?" (id 0) (at 118.11 88.7435 0))
+    (property "Reference" "U1" (id 0) (at 118.11 88.7435 0))
     (property "Value" "LP38692MPX-ADJ" (id 1) (at 118.11 91.5186 0))
     (property "Footprint" "Package_TO_SOT_SMD:SOT-223-5" (id 2) (at 118.11 87.63 0)
@@
   (symbol (lib_id "Device:C_Small") (at 97.79 100.33 0) (unit 1)
     (in_bom yes) (on_board yes)
-    (property "Reference" "C?" (id 0) (at 100.1268 99.1616 0)
+    (property "Reference" "C1" (id 0) (at 100.1268 99.1616 0)
       (effects (font (size 1.27 1.27)) (justify left))
     )

Commit message: Corrected PCB edge cuts, removed components
Will be mimicking layout done by Seth Sievers
Parts:
- renumbered C1 to C10, C2 to C11, J1 to J3, R1 to R4, R2 to R5, U1 to U4
Changed lines of the file:
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@@
   (symbol (lib_id "Data_Collection_KiCAD_Project-rescue:GND-power-Data_Collection_KiCAD_Project-rescue") (at 60.96 109.22 0) (unit 1)
     (in_bom yes) (on_board yes)
-    (property "Reference" "#PWR0112" (id 0) (at 60.96 115.57 0)
+    (property "Reference" "#PWR029" (id 0) (at 60.96 115.57 0)
       (effects (font (size 1.27 1.27)) hide)
     )
@@
   (symbol (lib_id "Data_Collection_KiCAD_Project-rescue:GND-power-Data_Collection_KiCAD_Project-rescue") (at 187.96 113.03 0) (unit 1)
     (in_bom yes) (on_board yes)
-    (property "Reference" "#PWR0114" (id 0) (at 187.96 119.38 0)
+    (property "Reference" "#PWR037" (id 0) (at 187.96 119.38 0)
       (effects (font (size 1.27 1.27)) hide)
     )
@@
   (symbol (lib_id "Data_Collection_KiCAD_Project-rescue:+5V-power-Data_Collection_KiCAD_Project-rescue") (at 187.96 92.71 0) (unit 1)
     (in_bom yes) (on_board yes)
-    (property "Reference" "#PWR0115" (id 0) (at 187.96 96.52 0)
+    (property "Reference" "#PWR036" (id 0) (at 187.96 96.52 0)
       (effects (font (size 1.27 1.27)) hide)
     )
@@
   (symbol (lib_id "dk_USB-DVI-HDMI-Connectors:10118192-0001LF") (at 50.8 100.33 0) (unit 1)
     (in_bom yes) (on_board yes)
-    (property "Reference" "J1" (id 0) (at 52.4256 81.407 0)
+    (property "Reference" "J3" (id 0) (at 52.4256 81.407 0)
       (effects (font (size 1.524 1.524)))
     )
@@
   (symbol (lib_id "Device:R_Small") (at 138.43 97.79 270) (unit 1)
     (in_bom yes) (on_board yes)
-    (property "Reference" "R2" (id 0) (at 139.5984 99.2886 0)
+    (property "Reference" "R5" (id 0) (at 139.5984 99.2886 0)
       (effects (font (size 1.27 1.27)) (justify left))
     )
@@
   (symbol (lib_id "Device:R_Small") (at 130.81 102.87 0) (unit 1)
     (in_bom yes) (on_board yes)
-    (property "Reference" "R1" (id 0) (at 132.3086 101.7016 0)
+    (property "Reference" "R4" (id 0) (at 132.3086 101.7016 0)
       (effects (font (size 1.27 1.27)) (justify left))
     )
@@
   (symbol (lib_id "power:GND") (at 97.79 102.87 0) (unit 1)
     (in_bom yes) (on_board yes)
-    (property "Reference" "#PWR0129" (id 0) (at 97.79 109.22 0)
+    (property "Reference" "#PWR030" (id 0) (at 97.79 109.22 0)
       (effects (font (size 1.27 1.27)) hide)
     )
@@
   (symbol (lib_id "power:+5V") (at 102.87 91.44 0) (unit 1)
     (in_bom yes) (on_board yes)
-    (property "Reference" "#PWR0113" (id 0) (at 102.87 95.25 0)
+    (property "Reference" "#PWR031" (id 0) (at 102.87 95.25 0)
       (effects (font (size 1.27 1.27)) hide)
     )
@@
   (symbol (lib_id "power:GND") (at 130.81 105.41 0) (unit 1)
     (in_bom yes) (on_board yes)
-    (property "Reference" "#PWR0132" (id 0) (at 130.81 111.76 0)
+    (property "Reference" "#PWR033" (id 0) (at 130.81 111.76 0)
       (effects (font (size 1.27 1.27)) hide)
     )
@@
   (symbol (lib_id "Device:C_Small") (at 144.78 102.87 0) (unit 1)
     (in_bom yes) (on_board yes)
-    (property "Reference" "C2" (id 0) (at 147.1168 101.7016 0)
+    (property "Reference" "C11" (id 0) (at 147.1168 101.7016 0)
       (effects (font (size 1.27 1.27)) (justify left))
     )
@@
   (symbol (lib_id "power:GND") (at 118.11 105.41 0) (unit 1)
     (in_bom yes) (on_board yes)
-    (property "Reference" "#PWR0130" (id 0) (at 118.11 111.76 0)
+    (property "Reference" "#PWR032" (id 0) (at 118.11 111.76 0)
       (effects (font (size 1.27 1.27)) hide)
     )
@@
   (symbol (lib_id "power:GND") (at 144.78 105.41 0) (unit 1)
     (in_bom yes) (on_board yes)
-    (property "Reference" "#PWR0133" (id 0) (at 144.78 111.76 0)
+    (property "Reference" "#PWR035" (id 0) (at 144.78 111.76 0)
       (effects (font (size 1.27 1.27)) hide)
     )
@@
   (symbol (lib_id "power:+3.3V") (at 133.35 91.44 0) (unit 1)
     (in_bom yes) (on_board yes)
-    (property "Reference" "#PWR0131" (id 0) (at 133.35 95.25 0)
+    (property "Reference" "#PWR034" (id 0) (at 133.35 95.25 0)
       (effects (font (size 1.27 1.27)) hide)
     )
@@
   (symbol (lib_id "Regulator_Linear:ADP7182AUJZ") (at 118.11 97.79 0) (mirror x) (unit 1)
     (in_bom yes) (on_board yes) (fields_autoplaced)
-    (property "Reference" "U1" (id 0) (at 118.11 88.7435 0))
+    (property "Reference" "U4" (id 0) (at 118.11 88.7435 0))
     (property "Value" "LP38692MPX-ADJ" (id 1) (at 118.11 91.5186 0))
     (property "Footprint" "Package_TO_SOT_SMD:SOT-223-5" (id 2) (at 118.11 87.63 0)
@@
   (symbol (lib_id "Device:C_Small") (at 97.79 100.33 0) (unit 1)
     (in_bom yes) (on_board yes)
-    (property "Reference" "C1" (id 0) (at 100.1268 99.1616 0)
-      (effects (font (size 1.27 1.27)) (justify left))
-    )
+    (property "Reference" "C10" (id 0) (at 100.1268 99.1616 0)
+      (effects (font (size 1.27 1.27)) (justify left))
+    )

Commit message: Organized components, arranged filter caps
Parts:
- J3: footprint Connector_USB:USB_Micro-B_Wuerth_614105150721_Vertical -> Connector_USB:USB_Micro-B_Molex-105017-0001
- R4, R5: footprint Resistor_SMD:R_0603_1608Metric_Pad1.05x0.95mm_HandSolder -> Resistor_SMD:R_0603_1608Metric_Pad0.98x0.95mm_HandSolder
Changed lines of the file:
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@@
       (effects (font (size 1.524 1.524)))
     )
-    (property "Footprint" "Connector_USB:USB_Micro-B_Wuerth_614105150721_Vertical" (id 2) (at 55.88 95.25 0)
+    (property "Footprint" "Connector_USB:USB_Micro-B_Molex-105017-0001" (id 2) (at 55.88 95.25 0)
       (effects (font (size 1.524 1.524)) (justify left) hide)
     )
@@
       (effects (font (size 1.27 1.27)) (justify left))
     )
-    (property "Footprint" "Resistor_SMD:R_0603_1608Metric_Pad1.05x0.95mm_HandSolder" (id 2) (at 138.43 97.79 0)
+    (property "Footprint" "Resistor_SMD:R_0603_1608Metric_Pad0.98x0.95mm_HandSolder" (id 2) (at 138.43 97.79 0)
       (effects (font (size 1.27 1.27)) hide)
     )
@@
       (effects (font (size 1.27 1.27)) (justify left))
     )
-    (property "Footprint" "Resistor_SMD:R_0603_1608Metric_Pad1.05x0.95mm_HandSolder" (id 2) (at 130.81 102.87 0)
+    (property "Footprint" "Resistor_SMD:R_0603_1608Metric_Pad0.98x0.95mm_HandSolder" (id 2) (at 130.81 102.87 0)
       (effects (font (size 1.27 1.27)) hide)
     )

Commit message: wtf is wrong with my github install
Connections:
- net +3V3: now also U4.3 (VOUT); no longer U4.5 (VOUT)
- net +5V: now also U4.1 (EN), U4.4 (VIN); no longer U4.2 (VIN), U4.3 (EN)
- net GND: now also U4.5 (GND); no longer U4.1 (GND)
- net at R4.1, R5.2: now also U4.2 (ADJ); no longer U4.4 (ADJ)
Changed lines of the file:
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@@
   (symbol (lib_id "Regulator_Linear:ADP7182AUJZ") (at 118.11 97.79 0) (mirror x) (unit 1)
     (in_bom yes) (on_board yes) (fields_autoplaced)
-    (property "Reference" "U4" (id 0) (at 118.11 88.7435 0))
-    (property "Value" "LP38692MPX-ADJ" (id 1) (at 118.11 91.5186 0))
-    (property "Footprint" "Package_TO_SOT_SMD:SOT-223-5" (id 2) (at 118.11 87.63 0)
+    (property "Reference" "U4" (id 0) (at 118.11 106.8365 0))
+    (property "Value" "LP38692MPX-ADJ" (id 1) (at 129.54 104.14 0))
+    (property "Footprint" "Package_TO_SOT_SMD:SOT-223-5" (id 2) (at 118.11 107.95 0)
       (effects (font (size 1.27 1.27) italic) hide)
     )
-    (property "Datasheet" "https://media.digikey.com/pdf/Data%20Sheets/Texas%20Instruments%20PDFs/LP38690,92-ADJ.pdf" (id 3) (at 118.11 85.09 0)
+    (property "Datasheet" "https://media.digikey.com/pdf/Data%20Sheets/Texas%20Instruments%20PDFs/LP38690,92-ADJ.pdf" (id 3) (at 118.11 110.49 0)
       (effects (font (size 1.27 1.27)) hide)
     )
