File: Hardware/COMPONENT_SHEETS/TEMPSENSOR_MIC184YMM.kicad_sch (KiCad schematic)
At the start: 2 parts

Commit message: I think it is done....
maybe

hopefully

please
Parts:
- gave numbers to parts that had none: 1
Changed lines of the file:
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@@
   (symbol (lib_id "MIC184YMM-TR:MIC184YMM-TR") (at 97.79 92.71 0) (unit 1)
     (in_bom yes) (on_board yes) (fields_autoplaced)
-    (property "Reference" "U?" (id 0) (at 129.0447 83.1245 0)
+    (property "Reference" "U6" (id 0) (at 129.0447 83.1245 0)
       (effects (font (size 1.524 1.524)))
     )
