File: Hardware/Data_Collection_KiCAD_Project.sch (KiCad schematic (older format))
At the start: 4 parts

Commit message: GPS layout change and test point tweaks
Parts:
- TP1, TP2, TP3, TP4: footprint Connector_PinHeader_1.00mm:PinHeader_1x01_P1.00mm_Vertical -> TestPoint:TestPoint_Loop_D1.80mm_Drill1.0mm_Beaded
Changed lines of the file:
@@
 F 0 "TP1" V 4400 1050 50  0000 C CNN
 F 1 "Debug Pad" V 4266 1197 50  0001 C CNN
-F 2 "Connector_PinHeader_1.00mm:PinHeader_1x01_P1.00mm_Vertical" H 4600 1350 60  0001 L CNN
+F 2 "TestPoint:TestPoint_Loop_D1.80mm_Drill1.0mm_Beaded" H 4600 1350 60  0001 L CNN
 F 3 "https://www.te.com/commerce/DocumentDelivery/DDEController?Action=srchrtrv&DocNm=1773266&DocType=DS&DocLang=English" H 4600 1450 60  0001 L CNN
 F 4 "A106144CT-ND" H 4600 1550 60  0001 L CNN "Digi-Key_PN"
@@
 F 0 "TP2" V 4400 1200 50  0000 C CNN
 F 1 "Debug Pad" V 4266 1347 50  0001 C CNN
-F 2 "Connector_PinHeader_1.00mm:PinHeader_1x01_P1.00mm_Vertical" H 4600 1500 60  0001 L CNN
+F 2 "TestPoint:TestPoint_Loop_D1.80mm_Drill1.0mm_Beaded" H 4600 1500 60  0001 L CNN
 F 3 "https://www.te.com/commerce/DocumentDelivery/DDEController?Action=srchrtrv&DocNm=1773266&DocType=DS&DocLang=English" H 4600 1600 60  0001 L CNN
 F 4 "A106144CT-ND" H 4600 1700 60  0001 L CNN "Digi-Key_PN"
@@
 F 0 "TP3" V 9950 1000 50  0000 C CNN
 F 1 "Debug Pad" V 9816 1147 50  0001 C CNN
-F 2 "Connector_PinHeader_1.00mm:PinHeader_1x01_P1.00mm_Vertical" H 10150 1300 60  0001 L CNN
+F 2 "TestPoint:TestPoint_Loop_D1.80mm_Drill1.0mm_Beaded" H 10150 1300 60  0001 L CNN
 F 3 "https://www.te.com/commerce/DocumentDelivery/DDEController?Action=srchrtrv&DocNm=1773266&DocType=DS&DocLang=English" H 10150 1400 60  0001 L CNN
 F 4 "A106144CT-ND" H 10150 1500 60  0001 L CNN "Digi-Key_PN"
@@
 F 0 "TP4" V 9950 1150 50  0000 C CNN
 F 1 "Debug Pad" V 9816 1297 50  0001 C CNN
-F 2 "Connector_PinHeader_1.00mm:PinHeader_1x01_P1.00mm_Vertical" H 10150 1450 60  0001 L CNN
+F 2 "TestPoint:TestPoint_Loop_D1.80mm_Drill1.0mm_Beaded" H 10150 1450 60  0001 L CNN
 F 3 "https://www.te.com/commerce/DocumentDelivery/DDEController?Action=srchrtrv&DocNm=1773266&DocType=DS&DocLang=English" H 10150 1550 60  0001 L CNN
 F 4 "A106144CT-ND" H 10150 1650 60  0001 L CNN "Digi-Key_PN"
@@
 Wire Wire Line
 	10150 1250 10050 1250
-Wire Bus Line
-	3250 1700 3250 1900
-Wire Bus Line
-	3250 4100 3250 4300
-Wire Bus Line
-	3250 5300 3250 5500
-Wire Bus Line
-	3250 5500 9400 5500
-Wire Bus Line
-	3250 4300 9400 4300
-Wire Bus Line
-	3250 2750 3250 3100
-Wire Bus Line
-	3250 3100 9400 3100
-Wire Bus Line
-	3250 1900 10900 1900
-Wire Bus Line
-	1150 3600 1150 7400
 $Sheet
 S 4650 1000 700  700
@@
 F12 "t_clk" I L 1550 6150 50
 $EndSheet
+Wire Bus Line
+	3250 1700 3250 1900
+Wire Bus Line
+	3250 4100 3250 4300
+Wire Bus Line
+	3250 5300 3250 5500
+Wire Bus Line
+	3250 5500 9400 5500
+Wire Bus Line
+	3250 4300 9400 4300
+Wire Bus Line
+	3250 2750 3250 3100
+Wire Bus Line
+	3250 3100 9400 3100
+Wire Bus Line
+	3250 1900 10900 1900
+Wire Bus Line
+	1150 3600 1150 7400
 $EndSCHEMATC

Commit message: routing progress and pin reassignment
Parts:
- removed TP4: Debug Pad, TestPoint:TestPoint_Loop_D1.80mm_Drill1.0mm_Beaded, symbol dk_Test-Points:RCT-0C
- TP1, TP2, TP3: footprint TestPoint:TestPoint_Loop_D1.80mm_Drill1.0mm_Beaded -> TestPoint:TestPoint_Pad_D1.0mm
Connections:
- no-connect marks 2 -> 3
Changed lines of the file:
@@
 F 0 "TP1" V 4400 1050 50  0000 C CNN
 F 1 "Debug Pad" V 4266 1197 50  0001 C CNN
-F 2 "TestPoint:TestPoint_Loop_D1.80mm_Drill1.0mm_Beaded" H 4600 1350 60  0001 L CNN
+F 2 "TestPoint:TestPoint_Pad_D1.0mm" H 4600 1350 60  0001 L CNN
 F 3 "https://www.te.com/commerce/DocumentDelivery/DDEController?Action=srchrtrv&DocNm=1773266&DocType=DS&DocLang=English" H 4600 1450 60  0001 L CNN
 F 4 "A106144CT-ND" H 4600 1550 60  0001 L CNN "Digi-Key_PN"
@@
 F 0 "TP2" V 4400 1200 50  0000 C CNN
 F 1 "Debug Pad" V 4266 1347 50  0001 C CNN
-F 2 "TestPoint:TestPoint_Loop_D1.80mm_Drill1.0mm_Beaded" H 4600 1500 60  0001 L CNN
+F 2 "TestPoint:TestPoint_Pad_D1.0mm" H 4600 1500 60  0001 L CNN
 F 3 "https://www.te.com/commerce/DocumentDelivery/DDEController?Action=srchrtrv&DocNm=1773266&DocType=DS&DocLang=English" H 4600 1600 60  0001 L CNN
 F 4 "A106144CT-ND" H 4600 1700 60  0001 L CNN "Digi-Key_PN"
@@
 F 0 "TP3" V 9950 1000 50  0000 C CNN
 F 1 "Debug Pad" V 9816 1147 50  0001 C CNN
-F 2 "TestPoint:TestPoint_Loop_D1.80mm_Drill1.0mm_Beaded" H 10150 1300 60  0001 L CNN
+F 2 "TestPoint:TestPoint_Pad_D1.0mm" H 10150 1300 60  0001 L CNN
 F 3 "https://www.te.com/commerce/DocumentDelivery/DDEController?Action=srchrtrv&DocNm=1773266&DocType=DS&DocLang=English" H 10150 1400 60  0001 L CNN
 F 4 "A106144CT-ND" H 10150 1500 60  0001 L CNN "Digi-Key_PN"
@@
 F 12 "Active" H 10150 2300 60  0001 L CNN "Status"
 	1    9950 1100
-	0    1    1    0
-$EndComp
-$Comp
-L dk_Test-Points:RCT-0C TP4
-U 1 1 61A902C0
-P 9950 1250
-F 0 "TP4" V 9950 1150 50  0000 C CNN
-F 1 "Debug Pad" V 9816 1297 50  0001 C CNN
-F 2 "TestPoint:TestPoint_Loop_D1.80mm_Drill1.0mm_Beaded" H 10150 1450 60  0001 L CNN
-F 3 "https://www.te.com/commerce/DocumentDelivery/DDEController?Action=srchrtrv&DocNm=1773266&DocType=DS&DocLang=English" H 10150 1550 60  0001 L CNN
-F 4 "A106144CT-ND" H 10150 1650 60  0001 L CNN "Digi-Key_PN"
-F 5 "RCT-0C" H 10150 1750 60  0001 L CNN "MPN"
-F 6 "Test and Measurement" H 10150 1850 60  0001 L CNN "Category"
-F 7 "Test Points" H 10150 1950 60  0001 L CNN "Family"
-F 8 "https://www.te.com/commerce/DocumentDelivery/DDEController?Action=srchrtrv&DocNm=1773266&DocType=DS&DocLang=English" H 10150 2050 60  0001 L CNN "DK_Datasheet_Link"
-F 9 "/product-detail/en/te-connectivity-amp-connectors/RCT-0C/A106144CT-ND/3477801" H 10150 2150 60  0001 L CNN "DK_Detail_Page"
-F 10 "PC TEST POINT NATURAL" H 10150 2250 60  0001 L CNN "Description"
-F 11 "TE Connectivity AMP Connectors" H 10150 2350 60  0001 L CNN "Manufacturer"
-F 12 "Active" H 10150 2450 60  0001 L CNN "Status"
-	1    9950 1250
 	0    1    1    0
 $EndComp
@@
 F12 "t_clk" I L 1550 6150 50
 $EndSheet
+NoConn ~ 10050 1250
 Wire Bus Line
 	3250 1700 3250 1900
